Commit message: updated UR5 descriptions

File: ws/src/ur5_description/robots/ur5.robot.urdf.xacro (robot description, xacro)
@@ -44,328 +44,330 @@
     </inertial>
   </xacro:macro>
-  <link name="world" />
-  <joint name="world_joint" type="fixed">
-    <parent link="world" />
-    <child link = "ur5_link_0" />
-    <origin xyz="0.0 0.0 0.0" rpy="0.0 0.0 0.0" />
-  </joint>
-  <link name="ur5_link_0" >
-    <visual>
-      <geometry>
-        <mesh filename="package://ur5_description/meshes/visual/link0.dae" />
-      </geometry>
-      <material name="LightGrey">
-        <color rgba="0.7 0.7 0.7 1.0"/>
-      </material>
-    </visual>
-    <collision>
-      <geometry>
-        <mesh filename="package://ur5_description/meshes/collision/link0.stl" />
-      </geometry>
-    </collision>
-    <xacro:cylinder_inertial radius="0.06" length="0.05" mass="${base_mass}">
-      <origin xyz="0.0 0.0 0.0" rpy="0 0 0" />
-    </xacro:cylinder_inertial>
-  </link>
-  <joint name="ur5_joint_1" type="revolute">
-    <parent link="ur5_link_0" />
-    <child link = "ur5_link_1" />
-    <origin xyz="0.0 0.0 ${shoulder_height}" rpy="0.0 0.0 0.0" />
-    <axis xyz="0 0 1" />
-    <limit lower="-3.14" upper="3.14" effort="150.0" velocity="3.15"/>
-    <dynamics damping="1" friction="1"/>
-  </joint>
-  <link name="ur5_link_1">
-    <visual>
-      <geometry>
-        <mesh filename="package://ur5_description/meshes/visual/link1.dae" />
-      </geometry>
-      <material name="LightGrey">
-        <color rgba="0.7 0.7 0.7 1.0"/>
-      </material>
-    </visual>
-    <collision>
-      <geometry>
-        <mesh filename="package://ur5_description/meshes/collision/link1.stl" />
-      </geometry>
-    </collision>
-    <xacro:cylinder_inertial radius="0.06" length="0.15" mass="${shoulder_mass}">
-      <origin xyz="0.0 0.0 0.0" rpy="0 0 0" />
-    </xacro:cylinder_inertial>
-  </link>
-  <joint name="ur5_joint_2" type="revolute">
-    <parent link="ur5_link_1" />
-    <child link = "ur5_link_2" />
-    <origin xyz="0.0 ${shoulder_offset} 0.0" rpy="0.0 ${pi / 2.0} 0.0" />
-    <axis xyz="0 1 0" />
-    <limit lower="-3.14" upper="3.14" effort="150.0" velocity="3.15"/>
-    <dynamics damping="1" friction="1"/>
-  </joint>
-  <link name="ur5_link_2">
-    <visual>
-      <geometry>
-        <mesh filename="package://ur5_description/meshes/visual/link2.dae" />
-      </geometry>
-      <material name="LightGrey">
-        <color rgba="0.7 0.7 0.7 1.0"/>
-      </material>
-    </visual>
-    <collision>
-      <geometry>
-        <mesh filename="package://ur5_description/meshes/collision/link2.stl" />
-      </geometry>
-    </collision>
-    <xacro:cylinder_inertial radius="0.06" length="0.56" mass="${upper_arm_mass}">
-      <origin xyz="0.0 0.0 0.28" rpy="0 0 0" />
-    </xacro:cylinder_inertial>
-  </link>
-  <joint name="ur5_joint_3" type="revolute">
-    <parent link="ur5_link_2" />
-    <child link = "ur5_link_3" />
-    <origin xyz="0.0 ${elbow_offset} ${upper_arm_length}" rpy="0.0 0.0 0.0" />
-    <axis xyz="0 1 0" />
-    <limit lower="-3.14" upper="3.14" effort="150.0" velocity="3.15"/>
-    <dynamics damping="1" friction="1"/>
-  </joint>
-  <link name="ur5_link_3">
-    <visual>
-      <geometry>
-        <mesh filename="package://ur5_description/meshes/visual/link3.dae" />
-      </geometry>
-      <material name="LightGrey">
-        <color rgba="0.7 0.7 0.7 1.0"/>
-      </material>
-    </visual>
-    <collision>
-      <geometry>
-        <mesh filename="package://ur5_description/meshes/collision/link3.stl" />
-      </geometry>
-    </collision>
-    <xacro:cylinder_inertial radius="0.06" length="0.5" mass="${forearm_mass}">
-      <origin xyz="0.0 0.0 0.25" rpy="0 0 0" />
-    </xacro:cylinder_inertial>
-  </link>
-  <joint name="ur5_joint_4" type="revolute">
-    <parent link="ur5_link_3" />
-    <child link = "ur5_link_4" />
-    <origin xyz="0.0 0.0 ${forearm_length}" rpy="0.0 ${pi / 2.0} 0.0" />
-    <axis xyz="0 1 0" />
-    <limit lower="-3.14" upper="3.14" effort="28.0" velocity="3.2"/>
-    <dynamics damping="1" friction="1"/>
-  </joint>
-  <link name="ur5_link_4">
-    <visual>
-      <geometry>
-        <mesh filename="package://ur5_description/meshes/visual/link4.dae" />
-      </geometry>
-      <material name="LightGrey">
-        <color rgba="0.7 0.7 0.7 1.0"/>
-      </material>
-    </visual>
-    <collision>
-      <geometry>
-        <mesh filename="package://ur5_description/meshes/collision/link4.stl" />
-      </geometry>
-    </collision>
-    <xacro:cylinder_inertial radius="0.6" length="0.12" mass="${wrist_1_mass}">
-      <origin xyz="0.0 0.0 0.0" rpy="0 0 0" />
-    </xacro:cylinder_inertial>
-  </link>
-  <joint name="ur5_joint_5" type="revolute">
-    <parent link="ur5_link_4" />
-    <child link = "ur5_link_5" />
-    <origin xyz="0.0 ${wrist_1_length} 0.0" rpy="0.0 0.0 0.0" />
-    <axis xyz="0 0 1" />
-    <limit lower="-3.14" upper="3.14" effort="28.0" velocity="3.2"/>
-    <dynamics damping="1" friction="1"/>
-  </joint>
-  <link name="ur5_link_5">
-    <visual>
-      <geometry>
-        <mesh filename="package://ur5_description/meshes/visual/link5.dae" />
-      </geometry>
-      <material name="LightGrey">
-        <color rgba="0.7 0.7 0.7 1.0"/>
-      </material>
-    </visual>
-    <collision>
-      <geometry>
-        <mesh filename="package://ur5_description/meshes/collision/link5.stl" />
-      </geometry>
-    </collision>
-    <xacro:cylinder_inertial radius="0.6" length="0.12" mass="${wrist_2_mass}">
-    <origin xyz="0.0 0.0 0.0" rpy="0 0 0" />
-    </xacro:cylinder_inertial>
-  </link>
-  <joint name="ur5_joint_6" type="revolute">
-    <parent link="ur5_link_5" />
-    <child link = "ur5_link_6" />
-    <origin xyz="0.0 0.0 ${wrist_2_length}" rpy="0.0 0.0 0.0" />
-    <axis xyz="0 1 0" />
-    <limit lower="-3.14" upper="3.14" effort="28.0" velocity="3.2"/>
-    <dynamics damping="1" friction="1"/>
-  </joint>
-  <link name="ur5_link_6">
-    <visual>
-      <geometry>
-        <mesh filename="package://ur5_description/meshes/visual/link6.dae" />
-      </geometry>
-      <material name="LightGrey">
-        <color rgba="0.7 0.7 0.7 1.0"/>
-      </material>
-    </visual>
-    <collision>
-      <geometry>
-        <mesh filename="package://ur5_description/meshes/collision/link6.stl" />
-      </geometry>
-    </collision>
-    <xacro:cylinder_inertial radius="0.6" length="0.12" mass="${wrist_3_mass}">
-      <origin xyz="0.0 0.0 0.0" rpy="0 0 0" />
-    </xacro:cylinder_inertial>
-  </link>
-  <joint name="ur5_ee_fixed_joint" type="fixed">
-    <parent link="ur5_link_6" />
-    <child link = "wsg_base" />
-    <origin xyz="0.0 ${wrist_3_length} 0.0" rpy="-${pi/2} 0.0 0.0" />
-  </joint>
-  <!-- This is where WSG50 begins -->
-  <link name="wsg_base">
-      <inertial>
-          <mass value="0.01" />
-          <origin xyz="0 0 0" />
-      	  <inertia ixx="0.01" ixy="0.0" ixz="0.0" iyy="0.01" iyz="0.0" izz="0.01" />
-      </inertial>
-      <visual>
-          <origin xyz="0.0 0 0" rpy="0 0 0" />
-          <geometry>
-             <mesh filename="package://ur5_description/meshes/visual/WSG50_110.stl" scale="1 1 1"/>
-          </geometry>
-          <material name="grey">
-		        <color rgba="0.5 0.5 0.5 1"/>
-      	  </material>
-      </visual>
-      <collision>
-          <origin xyz="0.0 0 0" rpy="0 0 0" />
-          <geometry>
-             <mesh filename="package://ur5_description/meshes/collision/WSG50_110.stl" scale="1 1 1"/>
-         </geometry>
-     </collision>
-  </link>
-  <joint name="joint_wsg_gripper_left" type="prismatic">
-     <limit lower="-0.055" upper="-0.0027" effort="100" velocity="100"/>
-     <origin xyz="0 0 0" rpy="0 0 0" />
-     <parent link="wsg_base"/>
-     <child link="wsg_gripper_left" />
-     <dynamics friction="1" damping="1" />
-     <axis xyz="1 0 0"/>
-  </joint>
-   <link name="wsg_gripper_left">
-      <inertial>
-          <mass value="0.01" />
-          <origin xyz="0 0 0" />
-          <inertia ixx="0.01" ixy="0.0" ixz="0.0" iyy="0.01" iyz="0.0" izz="0.01" />
-      </inertial>
-      <visual>
-          <origin xyz="0.0 0 0" rpy="0 0 0" />
-          <geometry>
-            <mesh filename="package://ur5_description/meshes/visual/GUIDE_WSG50_110.stl" scale="0.001 0.001 0.001"/>
-          </geometry>
-          <material name="black">
-            <color rgba="0 0 0 1"/>
-      	  </material>
-      </visual>
-      <collision>
-          <origin xyz="0 0 0" rpy="0 0 0" />
-          <geometry>
-             <mesh filename="package://ur5_description/meshes/collision/GUIDE_WSG50_110.stl" scale="0.001 0.001 0.001"/>
-          </geometry>
-      </collision>
-  </link>
-  <joint name="wsg_joint_finger_left" type="fixed">
-     <origin xyz="0 0 0.023" rpy="0 0 0" />
-     <parent link="wsg_gripper_left"/>
-     <child link="wsg_finger_left" />
-     <axis xyz="1 0 0"/>
-  </joint>
-  <link name="wsg_finger_left">
-      <inertial>
-          <mass value="0.01" />
-          <origin xyz="0 0 0" />
-          <inertia ixx="0.01" ixy="0.0" ixz="0.0" iyy="0.01" iyz="0.0" izz="0.01" />
-      </inertial>
-      <visual>
-          <origin xyz="0.0 0 0" rpy="0 0 0" />
-          <geometry>
-            <mesh filename="package://ur5_description/meshes/visual/WSG-FMF.stl" scale="0.001 0.001 0.001"/>
-          </geometry>
-          <material name="black">
-		        <color rgba="0 0 0 1"/>
-      	  </material>
-      </visual>
-      <collision>
-          <origin xyz="0 0 0" rpy="0 0 0" />
-          <geometry>
-             <mesh filename="package://ur5_description/meshes/collision/WSG-FMF.stl" scale="0.001 0.001 0.001"/>
-         </geometry>
-     </collision>
-  </link>
-  <joint name="joint_wsg_gripper_right" type="prismatic">
-     <limit lower="0.0027" upper="0.055" effort="100" velocity="100"/>
-     <origin xyz="0 0 0" rpy="0 0 3.14159" />
-     <parent link="wsg_base"/>
-     <child link="wsg_gripper_right" />
-     <axis xyz="-1 0 0"/>
-     <dynamics friction="1" damping="1" />
-  </joint>
-   <link name="wsg_gripper_right">
-      <inertial>
-          <mass value="0.01" />
-          <origin xyz="0 0 0" />
-          <inertia ixx="0.01" ixy="0.0" ixz="0.0" iyy="0.01" iyz="0.0" izz="0.01" />
-      </inertial>
-      <visual>
-          <origin xyz="0.0 0 0" rpy="0 0 0" />
-          <geometry>
-             <mesh filename="package://ur5_description/meshes/visual/GUIDE_WSG50_110.stl" scale="0.001 0.001 0.001"/>
-          </geometry>
-          <material name="black">
-	        	<color rgba="0 0 0 1"/>
-      	  </material>
-      </visual>
-      <collision>
-          <origin xyz="0 0 0" rpy="0 0 0" />
-          <geometry>
-             <mesh filename="package://ur5_description/meshes/collision/GUIDE_WSG50_110.stl" scale="0.001 0.001 0.001"/>
-         </geometry>
-      </collision>
-    </link>
-    <joint name="wsg_joint_finger_right" type="fixed">
-      <origin xyz="0 0 0.023" rpy="0 0 0" />
-      <parent link="wsg_gripper_right"/>
-      <child link="wsg_finger_right" />
-      <axis xyz="1 0 0"/>
-    </joint>
-    <link name="wsg_finger_right">
-      <inertial>
-          <mass value="0.01" />
-          <origin xyz="0 0 0" />
-          <inertia ixx="0.01" ixy="0.0" ixz="0.0" iyy="0.01" iyz="0.0" izz="0.01" />
-      </inertial>
-      <visual>
-          <origin xyz="0.0 0 0" rpy="0 0 0" />
-          <geometry>
-            <mesh filename="package://ur5_description/meshes/visual/WSG-FMF.stl" scale="0.001 0.001 0.001"/>
-          </geometry>
-          <material name="black">
-		        <color rgba="0 0 0 1"/>
-      	  </material>
-      </visual>
-      <collision>
-          <origin xyz="0 0 0" rpy="0 0 0" />
-          <geometry>
-            <mesh filename="package://ur5_description/meshes/collision/WSG-FMF.stl" scale="0.001 0.001 0.001"/>
-        </geometry>
-      </collision>
-    </link>
+  <xacro:macro name="ur5_arm" >
+	<link name="world" />
+	<joint name="world_joint" type="fixed">
+		<parent link="world" />
+		<child link = "ur5_link_0" />
+		<origin xyz="0.0 0.0 0.0" rpy="0.0 0.0 0.0" />
+	</joint>
+	<link name="ur5_link_0" >
+		<visual>
+		<geometry>
+			<mesh filename="package://ur5_description/meshes/visual/link0.dae" />
+		</geometry>
+		<material name="LightGrey">
+			<color rgba="0.7 0.7 0.7 1.0"/>
+		</material>
+		</visual>
+		<collision>
+		<geometry>
+			<mesh filename="package://ur5_description/meshes/collision/link0.stl" />
+		</geometry>
+		</collision>
+		<xacro:cylinder_inertial radius="0.06" length="0.05" mass="${base_mass}">
+		<origin xyz="0.0 0.0 0.0" rpy="0 0 0" />
+		</xacro:cylinder_inertial>
+	</link>
+	<joint name="ur5_joint_1" type="revolute">
+		<parent link="ur5_link_0" />
+		<child link = "ur5_link_1" />
+		<origin xyz="0.0 0.0 ${shoulder_height}" rpy="0.0 0.0 0.0" />
+		<axis xyz="0 0 1" />
+		<limit lower="-3.14" upper="3.14" effort="150.0" velocity="3.15"/>
+		<dynamics damping="1" friction="1"/>
+	</joint>
+	<link name="ur5_link_1">
+		<visual>
+		<geometry>
+			<mesh filename="package://ur5_description/meshes/visual/link1.dae" />
+		</geometry>
+		<material name="LightGrey">
+			<color rgba="0.7 0.7 0.7 1.0"/>
+		</material>
+		</visual>
+		<collision>
+		<geometry>
+			<mesh filename="package://ur5_description/meshes/collision/link1.stl" />
+		</geometry>
+		</collision>
+		<xacro:cylinder_inertial radius="0.06" length="0.15" mass="${shoulder_mass}">
+		<origin xyz="0.0 0.0 0.0" rpy="0 0 0" />
+		</xacro:cylinder_inertial>
+	</link>
+	<joint name="ur5_joint_2" type="revolute">
+		<parent link="ur5_link_1" />
+		<child link = "ur5_link_2" />
+		<origin xyz="0.0 ${shoulder_offset} 0.0" rpy="0.0 ${pi / 2.0} 0.0" />
+		<axis xyz="0 1 0" />
+		<limit lower="-3.14" upper="3.14" effort="150.0" velocity="3.15"/>
+		<dynamics damping="1" friction="1"/>
+	</joint>
+	<link name="ur5_link_2">
+		<visual>
+		<geometry>
+			<mesh filename="package://ur5_description/meshes/visual/link2.dae" />
+		</geometry>
+		<material name="LightGrey">
+			<color rgba="0.7 0.7 0.7 1.0"/>
+		</material>
+		</visual>
+		<collision>
+		<geometry>
+			<mesh filename="package://ur5_description/meshes/collision/link2.stl" />
+		</geometry>
+		</collision>
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