Commit message: implemented control + grip

File: ws/src/ur5_description/robots/ur5.transmission.xacro (robot description, xacro)
@@ -12,8 +12,8 @@
       <type>transmission_interface/SimpleTransmission</type>
       <joint name="ur5_joint1">
-        <hardwareInterface>hardware_interface/PositionJointInterface</hardwareInterface>
+        <hardwareInterface>hardware_interface/EffortJointInterface</hardwareInterface>
       </joint>
       <actuator name="ur5_motor1">
-        <hardwareInterface>hardware_interface/PositionJointInterface</hardwareInterface>
+        <hardwareInterface>hardware_interface/EffortJointInterface</hardwareInterface>
         <mechanicalReduction>1</mechanicalReduction>
       </actuator>
@@ -23,8 +23,8 @@
       <type>transmission_interface/SimpleTransmission</type>
       <joint name="ur5_joint2">
-        <hardwareInterface>hardware_interface/PositionJointInterface</hardwareInterface>
+        <hardwareInterface>hardware_interface/EffortJointInterface</hardwareInterface>
       </joint>
       <actuator name="ur5_motor2">
-        <hardwareInterface>hardware_interface/PositionJointInterface</hardwareInterface>
+        <hardwareInterface>hardware_interface/EffortJointInterface</hardwareInterface>
         <mechanicalReduction>1</mechanicalReduction>
       </actuator>
@@ -34,8 +34,8 @@
       <type>transmission_interface/SimpleTransmission</type>
       <joint name="ur5_joint3">
-        <hardwareInterface>hardware_interface/PositionJointInterface</hardwareInterface>
+        <hardwareInterface>hardware_interface/EffortJointInterface</hardwareInterface>
       </joint>
       <actuator name="ur5_motor3">
-        <hardwareInterface>hardware_interface/PositionJointInterface</hardwareInterface>
+        <hardwareInterface>hardware_interface/EffortJointInterface</hardwareInterface>
         <mechanicalReduction>1</mechanicalReduction>
       </actuator>
@@ -45,8 +45,8 @@
       <type>transmission_interface/SimpleTransmission</type>
       <joint name="ur5_joint4">
-        <hardwareInterface>hardware_interface/PositionJointInterface</hardwareInterface>
+        <hardwareInterface>hardware_interface/EffortJointInterface</hardwareInterface>
       </joint>
       <actuator name="ur5_motor4">
-        <hardwareInterface>hardware_interface/PositionJointInterface</hardwareInterface>
+        <hardwareInterface>hardware_interface/EffortJointInterface</hardwareInterface>
         <mechanicalReduction>1</mechanicalReduction>
       </actuator>
@@ -56,8 +56,8 @@
       <type>transmission_interface/SimpleTransmission</type>
       <joint name="ur5_joint5">
-        <hardwareInterface>hardware_interface/PositionJointInterface</hardwareInterface>
+        <hardwareInterface>hardware_interface/EffortJointInterface</hardwareInterface>
       </joint>
       <actuator name="ur5_motor5">
-        <hardwareInterface>hardware_interface/PositionJointInterface</hardwareInterface>
+        <hardwareInterface>hardware_interface/EffortJointInterface</hardwareInterface>
         <mechanicalReduction>1</mechanicalReduction>
       </actuator>
@@ -67,8 +67,8 @@
       <type>transmission_interface/SimpleTransmission</type>
       <joint name="ur5_joint6">
-        <hardwareInterface>hardware_interface/PositionJointInterface</hardwareInterface>
+        <hardwareInterface>hardware_interface/EffortJointInterface</hardwareInterface>
       </joint>
       <actuator name="ur5_motor6">
-        <hardwareInterface>hardware_interface/PositionJointInterface</hardwareInterface>
+        <hardwareInterface>hardware_interface/EffortJointInterface</hardwareInterface>
         <mechanicalReduction>1</mechanicalReduction>
       </actuator>

File: ws/src/ur5_description/robots/ur5.urdf.xacro (robot description, xacro)
@@ -2,13 +2,14 @@
 <robot xmlns:xacro="http://www.ros.org/wiki/xacro" name="ur5">
   <!-- load arm + hand -->
-  <xacro:include filename="$(find ur5_description)/robots/ur5_arm.xacro" />
-  <!-- <xacro:include filename="$(find ur5_description)/robots/ur5_gripper.xacro" /> -->
+  <xacro:include filename="$(find ur5_description)/robots/ur5_arm.xacro"/>
+  <!-- <xacro:include filename="$(find ur5_description)/robots/ur5_gripper.xacro"/> -->
   <!-- load gazebo + transmission files -->
-  <xacro:include filename="$(find ur5_description)/robots/ur5.gazebo.xacro" />
-  <xacro:include filename="$(find ur5_description)/robots/ur5.transmission.xacro" />
+  <xacro:include filename="$(find ur5_description)/robots/ur5.gazebo.xacro"/>
+  <xacro:include filename="$(find ur5_description)/robots/ur5.transmission.xacro"/>
+  <link name="world"/>
   <!-- construct robot -->
-  <xacro:ur5_arm />
-  <!-- <xacro:ur5_gripper /> -->
-  <xacro:ur5_gazebo />
-  <xacro:ur5_transmission />
+  <xacro:ur5_arm/>
+  <!-- <xacro:ur5_gripper/> -->
+  <xacro:ur5_gazebo/>
+  <xacro:ur5_transmission/>
 </robot>

File: ws/src/ur5_description/robots/ur5_arm.xacro (robot description, xacro)
@@ -2,42 +2,42 @@
 <robot xmlns:xacro="http://www.ros.org/wiki/xacro" name="ur5">
   <!-- properties of the UR5 robot -->
-  <xacro:property name="base_mass" value="0.1" />
-  <xacro:property name="shoulder_mass" value="0.1" />
-  <xacro:property name="upper_arm_mass" value="0.1" />
-  <xacro:property name="forearm_mass" value="0.1" />
-  <xacro:property name="wrist_1_mass" value="0.1" />
-  <xacro:property name="wrist_2_mass" value="0.1" />
-  <xacro:property name="wrist_3_mass" value="0.1" />
-  <xacro:property name="shoulder_cog" value="0.0 0.00193 -0.02561" />
-  <xacro:property name="upper_arm_cog" value="0.0 -0.024201 0.2125" />
-  <xacro:property name="forearm_cog" value="0.0 0.0265 0.11993" />
-  <xacro:property name="wrist_1_cog" value="0.0 0.110949 0.01634" />
-  <xacro:property name="wrist_2_cog" value="0.0 0.0018 0.11099" />
-  <xacro:property name="wrist_3_cog" value="0.0 0.001159 0.0" />
-  <xacro:property name="ur5_d1" value="0.089159" />
-  <xacro:property name="ur5_a2" value="-0.42500" />
-  <xacro:property name="ur5_a3" value="-0.39225" />
-  <xacro:property name="ur5_d4" value="0.14215" />
-  <xacro:property name="ur5_d5" value="0.1" />
-  <xacro:property name="ur5_d6" value="0.0983" />
-  <xacro:property name="shoulder_offset" value="0.13585" />
-  <xacro:property name="elbow_offset" value="-0.1197" />
-  <xacro:property name="shoulder_height" value="${ur5_d1}" />
-  <xacro:property name="upper_arm_length" value="${-ur5_a2}" />
-  <xacro:property name="forearm_length" value="${-ur5_a3}" />
-  <xacro:property name="wrist_1_length" value="${ur5_d4 - elbow_offset - shoulder_offset}" />
-  <xacro:property name="wrist_2_length" value="${ur5_d5}" />
-  <xacro:property name="wrist_3_length" value="${ur5_d6}" />
-  <xacro:property name="shoulder_radius" value="0.060" />
-  <xacro:property name="upper_arm_radius" value="0.054" />
-  <xacro:property name="elbow_radius" value="0.060" />
-  <xacro:property name="forearm_radius" value="0.040" />
-  <xacro:property name="wrist_radius" value="0.045" />
+  <xacro:property name="base_mass" value="0.1"/>
+  <xacro:property name="shoulder_mass" value="0.1"/>
+  <xacro:property name="upper_arm_mass" value="0.1"/>
+  <xacro:property name="forearm_mass" value="0.1"/>
+  <xacro:property name="wrist_1_mass" value="0.1"/>
+  <xacro:property name="wrist_2_mass" value="0.1"/>
+  <xacro:property name="wrist_3_mass" value="0.1"/>
+  <xacro:property name="shoulder_cog" value="0.0 0.00193 -0.02561"/>
+  <xacro:property name="upper_arm_cog" value="0.0 -0.024201 0.2125"/>
+  <xacro:property name="forearm_cog" value="0.0 0.0265 0.11993"/>
+  <xacro:property name="wrist_1_cog" value="0.0 0.110949 0.01634"/>
+  <xacro:property name="wrist_2_cog" value="0.0 0.0018 0.11099"/>
+  <xacro:property name="wrist_3_cog" value="0.0 0.001159 0.0"/>
+  <xacro:property name="ur5_d1" value="0.089159"/>
+  <xacro:property name="ur5_a2" value="-0.42500"/>
+  <xacro:property name="ur5_a3" value="-0.39225"/>
+  <xacro:property name="ur5_d4" value="0.14215"/>
+  <xacro:property name="ur5_d5" value="0.1"/>
+  <xacro:property name="ur5_d6" value="0.0983"/>
+  <xacro:property name="shoulder_offset" value="0.13585"/>
+  <xacro:property name="elbow_offset" value="-0.1197"/>
+  <xacro:property name="shoulder_height" value="${ur5_d1}"/>
+  <xacro:property name="upper_arm_length" value="${-ur5_a2}"/>
+  <xacro:property name="forearm_length" value="${-ur5_a3}"/>
+  <xacro:property name="wrist_1_length" value="${ur5_d4 - elbow_offset - shoulder_offset}"/>
+  <xacro:property name="wrist_2_length" value="${ur5_d5}"/>
+  <xacro:property name="wrist_3_length" value="${ur5_d6}"/>
+  <xacro:property name="shoulder_radius" value="0.060"/>
+  <xacro:property name="upper_arm_radius" value="0.054"/>
+  <xacro:property name="elbow_radius" value="0.060"/>
+  <xacro:property name="forearm_radius" value="0.040"/>
+  <xacro:property name="wrist_radius" value="0.045"/>
   <!-- cyldenrical inertia for approximation for the link inertias -->
   <!-- <xacro:macro name="cylinder_inertial" params="radius length mass *origin">
     <inertial>
-      <mass value="${0.01 />
-      <insert_block name="origin" />
-      <inertia ixx="${0.0833333 * mass * (3 * radius * radius + length * length)}" ixy="0.0" ixz="0.0" iyy="${0.0833333 * mass * (3 * radius * radius + length * length)}" iyz="0.0" izz="${0.5 * mass * radius * radius}" />
+      <mass value="${0.01/>
+      <insert_block name="origin"/>
+      <inertia ixx="${0.0833333 * mass * (3 * radius * radius + length * length)}" ixy="0.0" ixz="0.0" iyy="${0.0833333 * mass * (3 * radius * radius + length * length)}" iyz="0.0" izz="${0.5 * mass * radius * radius}"/>
     </inertial>
   </xacro:macro> -->
@@ -52,7 +52,7 @@
     <!-- fix the robot to the Gazebo world coordinate system -->
     <joint name="world_to_robot" type="fixed">
-      <origin xyz="0.0 0.0 0.2" rpy="0.0 0.0 0.0" />
-      <parent link="world" />
-      <child link="ur5_link0" />
+      <origin xyz="0.0 0.0 0.0" rpy="0.0 0.0 0.0"/>
+      <parent link="world"/>
+      <child link="ur5_link0"/>
     </joint>
     <!-- link 0 -->
@@ -61,20 +61,20 @@
       <visual>
         <geometry>
-          <mesh filename="package://ur5_description/meshes/visual/link0.dae" />
-        </geometry>
-        <material name="LightGrey">
-          <color rgba="0.7 0.7 0.7 1.0" />
-        </material>
-      </visual>
-      <collision>
-        <geometry>
-          <mesh filename="package://ur5_description/meshes/collision/link0.stl" />
+          <mesh filename="package://ur5_description/meshes/visual/link0.dae"/>
+        </geometry>
+        <material name="LightGrey">
+          <color rgba="0.7 0.7 0.7 1.0"/>
+        </material>
+      </visual>
+      <collision>
+        <geometry>
+          <mesh filename="package://ur5_description/meshes/collision/link0.stl"/>
         </geometry>
       </collision>
       <!-- <cylinder_inertial radius="0.06" length="0.05" mass="${base_mass}">
-        <origin xyz="0.0 0.0 0.0" rpy="0 0 0" />
-      </cylinder_inertial> -->
-      <inertial>
-        <mass value="0.01"/>
+        <origin xyz="0.0 0.0 0.0" rpy="0 0 0"/>
+      </cylinder_inertial> -->
+      <inertial>
+        <mass value="10.0"/>
         <inertia ixx="0.004433" ixy="0.0" ixz="0.0" iyy="0.00443333156" iyz="0.0" izz="0.0072"/>
       </inertial>
@@ -82,10 +82,10 @@
     <!-- joint1 connects link0 and link1 -->
     <joint name="ur5_joint1" type="revolute">
-      <parent link="ur5_link0" />
-      <child link="ur5_link1" />
-      <origin xyz="0.0 0.0 ${shoulder_height}" rpy="0.0 0.0 0.0" />
-      <axis xyz="0 0 1" />
-      <!-- <limit lower="-3.14" upper="3.14" effort="150.0" velocity="3.15" /> -->
-      <limit lower="${-pi}" upper="${pi}" effort="150.0" velocity="${pi}"/>
+      <parent link="ur5_link0"/>
+      <child link="ur5_link1"/>
+      <origin xyz="0.0 0.0 ${shoulder_height}" rpy="0.0 0.0 0.0"/>
+      <axis xyz="0 0 1"/>
+      <!-- <limit lower="-3.14" upper="3.14" effort="112.0" velocity="3.15"/> -->
+      <limit lower="${-pi}" upper="${pi}" effort="112.0" velocity="${pi}"/>
       <dynamics damping="0.4" friction="0.0"/>
     </joint>
@@ -95,20 +95,20 @@
       <visual>
         <geometry>
-          <mesh filename="package://ur5_description/meshes/visual/link1.dae" />
-        </geometry>
-        <material name="LightGrey">
-          <color rgba="0.7 0.7 0.7 1.0" />
-        </material>
-      </visual>
-      <collision>
-        <geometry>
-          <mesh filename="package://ur5_description/meshes/collision/link1.stl" />
+          <mesh filename="package://ur5_description/meshes/visual/link1.dae"/>
+        </geometry>
+        <material name="LightGrey">
+          <color rgba="0.7 0.7 0.7 1.0"/>
+        </material>
+      </visual>
+      <collision>
+        <geometry>
+          <mesh filename="package://ur5_description/meshes/collision/link1.stl"/>
         </geometry>
       </collision>
       <!-- <cylinder_inertial radius="0.06" length="0.15" mass="${shoulder_mass}">
-        <origin xyz="0.0 0.0 0.0" rpy="0 0 0" />
-      </cylinder_inertial> -->
-      <inertial>
-        <mass value="0.01"/>
+        <origin xyz="0.0 0.0 0.0" rpy="0 0 0"/>
+      </cylinder_inertial> -->
+      <inertial>
+        <mass value="3.7"/>
         <inertia ixx="0.010267495893" ixy="0.0" ixz="0.0" iyy="0.010267495893" iyz="0.0" izz="0.00666"/>
         <origin rpy="0.0 0.0 0.0" xyz="0.0 0.00193 -0.02561"/>
@@ -117,10 +117,10 @@
     <!-- joint2 connects link1 and link2 -->
     <joint name="ur5_joint2" type="revolute">
-      <parent link="ur5_link1" />
-      <child link="ur5_link2" />
-      <origin xyz="0.0 ${shoulder_offset} 0.0" rpy="0.0 ${pi / 2.0} 0.0" />
-      <axis xyz="0 1 0" />
-      <!-- <limit lower="-3.14" upper="3.14" effort="150.0" velocity="3.15" /> -->
-      <limit lower="${-pi}" upper="${pi}" effort="150.0" velocity="${pi}"/>
+      <parent link="ur5_link1"/>
+      <child link="ur5_link2"/>
+      <origin xyz="0.0 ${shoulder_offset} 0.0" rpy="0.0 ${pi / 2.0} 0.0"/>
+      <axis xyz="0 1 0"/>
+      <!-- <limit lower="-3.14" upper="3.14" effort="112.0" velocity="3.15"/> -->
+      <limit lower="${-pi}" upper="${pi}" effort="112.0" velocity="${pi}"/>
       <dynamics damping="0.4" friction="0.0"/>
     </joint>
@@ -130,21 +130,21 @@
       <visual>
         <geometry>
-          <mesh filename="package://ur5_description/meshes/visual/link2.dae" />
-        </geometry>
-        <material name="LightGrey">
-          <color rgba="0.7 0.7 0.7 1.0" />
-        </material>
-      </visual>
-      <collision>
-        <geometry>
-          <mesh filename="package://ur5_description/meshes/collision/link2.stl" />
+          <mesh filename="package://ur5_description/meshes/visual/link2.dae"/>
+        </geometry>
+        <material name="LightGrey">
+          <color rgba="0.7 0.7 0.7 1.0"/>
+        </material>
+      </visual>
+      <collision>
+        <geometry>
+          <mesh filename="package://ur5_description/meshes/collision/link2.stl"/>
         </geometry>
       </collision>
       <!-- <cylinder_inertial radius="0.06" length="0.56" mass="${upper_arm_mass}">
-        <origin xyz="0.0 0.0 0.28" rpy="0 0 0" />
-      </cylinder_inertial> -->
-      <inertial>
-        <mass value="0.01"/>
-        <inertia ixx="0.22689067591036" ixy="0.0" ixz="0.0" iyy="0.22689067591036" iyz="0.0" izz="0.0151074" />
+        <origin xyz="0.0 0.0 0.28" rpy="0 0 0"/>
+      </cylinder_inertial> -->
+      <inertial>
+        <mass value="8.393"/>
+        <inertia ixx="0.22689067591036" ixy="0.0" ixz="0.0" iyy="0.22689067591036" iyz="0.0" izz="0.0151074"/>
         <origin rpy="0.0 0.0 0.0" xyz="0.0 -0.024201 0.2125"/>
       </inertial>
@@ -152,11 +152,11 @@
     <!-- joint3 connects link2 and link3 -->
     <joint name="ur5_joint3" type="revolute">
-      <parent link="ur5_link2" />
-      <child link="ur5_link3" />
-      <origin xyz="0.0 ${elbow_offset} ${upper_arm_length}" rpy="0.0 0.0 0.0" />
-      <axis xyz="0 1 0" />
-      <!-- <limit lower="-3.14" upper="3.14" effort="150.0" velocity="3.15" /> -->
-      <limit lower="${-pi}" upper="${pi}" effort="150.0" velocity="${pi}" />
-	  <dynamics damping="0.4" friction="0.0" />
+      <parent link="ur5_link2"/>
+      <child link="ur5_link3"/>
+      <origin xyz="0.0 ${elbow_offset} ${upper_arm_length}" rpy="0.0 0.0 0.0"/>
+      <axis xyz="0 1 0"/>
+      <!-- <limit lower="-3.14" upper="3.14" effort="112.0" velocity="3.15"/> -->
+      <limit lower="${-pi}" upper="${pi}" effort="112.0" velocity="${pi}"/>
+	  <dynamics damping="0.4" friction="0.0"/>
     </joint>
     <!-- link 3 -->
@@ -165,31 +165,31 @@
       <visual>
         <geometry>
-          <mesh filename="package://ur5_description/meshes/visual/link3.dae" />
-        </geometry>
-        <material name="LightGrey">
-          <color rgba="0.7 0.7 0.7 1.0" />
-        </material>
-      </visual>
-      <collision>
-        <geometry>
-          <mesh filename="package://ur5_description/meshes/collision/link3.stl" />
+          <mesh filename="package://ur5_description/meshes/visual/link3.dae"/>
+        </geometry>
+        <material name="LightGrey">
+          <color rgba="0.7 0.7 0.7 1.0"/>
+        </material>
+      </visual>
+      <collision>
+        <geometry>
+          <mesh filename="package://ur5_description/meshes/collision/link3.stl"/>
         </geometry>
       </collision>
       <!-- <cylinder_inertial radius="0.06" length="0.5" mass="${forearm_mass}">
-        <origin xyz="0.0 0.0 0.25" rpy="0 0 0" />
-      </cylinder_inertial> -->
-      <inertial>
-        <mass value="0.01"/>
+        <origin xyz="0.0 0.0 0.25" rpy="0 0 0"/>
+      </cylinder_inertial> -->
+      <inertial>
+        <mass value="2.33"/>
         <origin rpy="0.0 0.0 0.0" xyz="0.0 0.0265 0.11993"/>
-        <inertia ixx="0.049443313556" ixy="0.0" ixz="0.0" iyy="0.049443313556" iyz="0.0" izz="0.004095" />
+        <inertia ixx="0.049443313556" ixy="0.0" ixz="0.0" iyy="0.049443313556" iyz="0.0" izz="0.004095"/>
       </inertial>
     </link>
     <!-- joint4 connects link3 and link4 -->
     <joint name="ur5_joint4" type="revolute">
-      <parent link="ur5_link3" />
-      <child link="ur5_link4" />
-      <origin xyz="0.0 0.0 ${forearm_length}" rpy="0.0 ${pi / 2.0} 0.0" />
-      <axis xyz="0 1 0" />
-      <!-- <limit lower="-3.14" upper="3.14" effort="28.0" velocity="3.2" /> -->
+      <parent link="ur5_link3"/>
+      <child link="ur5_link4"/>
+      <origin xyz="0.0 0.0 ${forearm_length}" rpy="0.0 ${pi / 2.0} 0.0"/>
+      <axis xyz="0 1 0"/>
+      <!-- <limit lower="-3.14" upper="3.14" effort="28.0" velocity="3.2"/> -->
       <limit lower="${-1.0 * pi}" upper="${0.25 * pi}" effort="28.0" velocity="${pi}"/>
       <dynamics damping="0.3" friction="0.0"/>
@@ -199,31 +199,31 @@
       <visual>
         <geometry>
-          <mesh filename="package://ur5_description/meshes/visual/link4.dae" />
-        </geometry>
-        <material name="LightGrey">
-          <color rgba="0.7 0.7 0.7 1.0" />
-        </material>
-      </visual>
-      <collision>
-        <geometry>
-          <mesh filename="package://ur5_description/meshes/collision/link4.stl" />
+          <mesh filename="package://ur5_description/meshes/visual/link4.dae"/>
+        </geometry>
+        <material name="LightGrey">
+          <color rgba="0.7 0.7 0.7 1.0"/>
+        </material>
+      </visual>
+      <collision>
+        <geometry>
+          <mesh filename="package://ur5_description/meshes/collision/link4.stl"/>
         </geometry>
       </collision>
       <!-- <cylinder_inertial radius="0.6" length="0.12" mass="${wrist_1_mass}">
-        <origin xyz="0.0 0.0 0.0" rpy="0 0 0" />
-      </cylinder_inertial> -->
-      <inertial>
-        <mass value="0.01"/>
+        <origin xyz="0.0 0.0 0.0" rpy="0 0 0"/>
+      </cylinder_inertial> -->
+      <inertial>
+        <mass value="1.219"/>
         <origin rpy="0.0 0.0 0.0" xyz="0.0 0.110949 0.01634"/>
-        <inertia ixx="0.11117275553088" ixy="0.0" ixz="0.0" iyy="0.11117275553088" iyz="0.0" izz="0.21942" />
+        <inertia ixx="0.11117275553088" ixy="0.0" ixz="0.0" iyy="0.11117275553088" iyz="0.0" izz="0.21942"/>
       </inertial>
     </link>
     <!-- joint5 connects link4 and link5 -->
     <joint name="ur5_joint5" type="revolute">
-      <parent link="ur5_link4" />
-      <child link="ur5_link5" />
-      <origin xyz="0.0 ${wrist_1_length} 0.0" rpy="0.0 0.0 0.0" />
-      <axis xyz="0 0 1" />
-      <!-- <limit lower="-3.14" upper="3.14" effort="28.0" velocity="3.2" /> -->
+      <parent link="ur5_link4"/>
+      <child link="ur5_link5"/>
+      <origin xyz="0.0 ${wrist_1_length} 0.0" rpy="0.0 0.0 0.0"/>
+      <axis xyz="0 0 1"/>
+      <!-- <limit lower="-3.14" upper="3.14" effort="28.0" velocity="3.2"/> -->
       <limit lower="${-1.0 * pi}" upper="${1.0 * pi}" effort="28.0" velocity="${pi}"/>
       <dynamics damping="0.3" friction="0.0"/>
@@ -233,31 +233,31 @@
       <visual>
         <geometry>
-          <mesh filename="package://ur5_description/meshes/visual/link5.dae" />
-        </geometry>
-        <material name="LightGrey">
-          <color rgba="0.7 0.7 0.7 1.0" />
-        </material>
-      </visual>
-      <collision>
-        <geometry>
-          <mesh filename="package://ur5_description/meshes/collision/link5.stl" />
+          <mesh filename="package://ur5_description/meshes/visual/link5.dae"/>
+        </geometry>
+        <material name="LightGrey">
+          <color rgba="0.7 0.7 0.7 1.0"/>
+        </material>
+      </visual>
+      <collision>
+        <geometry>
+          <mesh filename="package://ur5_description/meshes/collision/link5.stl"/>
         </geometry>
       </collision>
       <!-- <cylinder_inertial radius="0.6" length="0.12" mass="${wrist_2_mass}">
-        <origin xyz="0.0 0.0 0.0" rpy="0 0 0" />
-      </cylinder_inertial> -->
-      <inertial>
-        <mass value="0.01"/>
+        <origin xyz="0.0 0.0 0.0" rpy="0 0 0"/>
+      </cylinder_inertial> -->
+      <inertial>
+        <mass value="1.219"/>
         <origin rpy="0.0 0.0 0.0" xyz="0.0 0.0018 0.11099"/>
-        <inertia ixx="0.11117275553088" ixy="0.0" ixz="0.0" iyy="0.11117275553088" iyz="0.0" izz="0.21942" />
+        <inertia ixx="0.11117275553088" ixy="0.0" ixz="0.0" iyy="0.11117275553088" iyz="0.0" izz="0.21942"/>
       </inertial>
     </link>
     <!-- joint6 connects link5 and link6 -->
     <joint name="ur5_joint6" type="revolute">
-      <parent link="ur5_link5" />
-      <child link="ur5_link6" />
-      <origin xyz="0.0 0.0 ${wrist_2_length}" rpy="0.0 0.0 0.0" />
-      <axis xyz="0 1 0" />
-      <!-- <limit lower="-3.14" upper="3.14" effort="28.0" velocity="3.2" /> -->
+      <parent link="ur5_link5"/>
+      <child link="ur5_link6"/>
+      <origin xyz="0.0 0.0 ${wrist_2_length}" rpy="0.0 0.0 0.0"/>
+      <axis xyz="0 1 0"/>
+      <!-- <limit lower="-3.14" upper="3.14" effort="28.0" velocity="3.2"/> -->
       <limit lower="${-1.0 * pi}" upper="${1.0 * pi}" effort="28.0" velocity="${pi}"/>
       <dynamics damping="0.3" friction="0.0"/>
@@ -267,31 +267,30 @@
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