Commit message: implemented control + grip

File: ws/src/ur5_description/robots/ur5_with_wsg.urdf.xacro (robot description, xacro)
@@ -2,16 +2,16 @@
 <robot xmlns:xacro="http://www.ros.org/wiki/xacro" name="ur5">
     <!-- load arm -->
-    <xacro:include filename="$(find ur5_description)/robots/ur5_arm.xacro" />
-    <xacro:include filename="$(find ur5_description)/robots/ur5.gazebo.xacro" />
-    <xacro:include filename="$(find ur5_description)/robots/ur5.transmission.xacro" />
+    <xacro:include filename="$(find ur5_description)/robots/ur5_arm.xacro"/>
+    <xacro:include filename="$(find ur5_description)/robots/ur5.gazebo.xacro"/>
+    <xacro:include filename="$(find ur5_description)/robots/ur5.transmission.xacro"/>
     <!-- load end-effector -->
     <xacro:include filename="$(find ur5_description)/robots/wsg.gazebo.xacro"/>
-    <xacro:include filename="$(find ur5_description)/robots/wsg.transmission.xacro" />
-    <xacro:include filename="$(find ur5_description)/robots/wsg.xacro" />
+    <xacro:include filename="$(find ur5_description)/robots/wsg.transmission.xacro"/>
+    <xacro:include filename="$(find ur5_description)/robots/wsg.xacro"/>
     <link name="world"/>
     <!-- construct robot note: make a variable to move the robot -->
-    <xacro:ur5_arm />
-    <xacro:ur5_gazebo />
-    <xacro:ur5_transmission />
+    <xacro:ur5_arm/>
+    <xacro:ur5_gazebo/>
+    <xacro:ur5_transmission/>
     <!-- construct end effector -->
     <xacro:wsg/>

File: ws/src/ur5_description/robots/wsg.gazebo.xacro (robot description, xacro)
@@ -5,44 +5,48 @@
     <gazebo reference="wsg_base">
       <selfCollide>true</selfCollide>
-      <mu1>0.1</mu1>
-      <mu2>0.1</mu2>
+      <mu1>1</mu1>
+      <mu2>1</mu2>
       <material>Gazebo/Grey</material>
     </gazebo>
-    <!-- Right -->
+    <!-- right -->
     <gazebo reference="wsg_finger_mount_right">
       <selfCollide>true</selfCollide>
-      <mu1>0.1</mu1>
-      <mu2>0.1</mu2>
+      <mu1>1</mu1>
+      <mu2>1</mu2>
       <material>Gazebo/Grey</material>
     </gazebo>
     <gazebo reference="wsg_finger_right">
       <selfCollide>true</selfCollide>
-      <mu1>0.1</mu1>
-      <mu2>0.1</mu2>
+      <mu1>1</mu1>
+      <mu2>1</mu2>
       <material>Gazebo/Black</material>
     </gazebo>
     <gazebo reference="wsg_fingertip_right">
       <selfCollide>true</selfCollide>
-      <mu1>0.1</mu1>
-      <mu2>0.1</mu2>
+      <mu1>1</mu1>
+      <mu2>1</mu2>
       <material>Gazebo/Blue</material>
     </gazebo>
-    <!-- Left -->
+    <gazebo reference="wsg_base_mount_right_joint">
+      <implicitSpringDamper>1</implicitSpringDamper>
+      <provideFeedback>true</provideFeedback>
+    </gazebo>
+    <!-- left -->
     <gazebo reference="wsg_finger_mount_left">
       <selfCollide>true</selfCollide>
-      <mu1>0.1</mu1>
-      <mu2>0.1</mu2>
+      <mu1>1</mu1>
+      <mu2>1</mu2>
       <material>Gazebo/Grey</material>
     </gazebo>
     <gazebo reference="wsg_finger_left">
       <selfCollide>true</selfCollide>
-      <mu1>0.1</mu1>
-      <mu2>0.1</mu2>
+      <mu1>1</mu1>
+      <mu2>1</mu2>
       <material>Gazebo/Black</material>
     </gazebo>
     <gazebo reference="wsg_fingertip_left">
       <selfCollide>true</selfCollide>
-      <mu1>0.1</mu1>
-      <mu2>0.1</mu2>
+      <mu1>1</mu1>
+      <mu2>1</mu2>
       <material>Gazebo/Blue</material>
     </gazebo>
@@ -51,8 +55,4 @@
       <provideFeedback>true</provideFeedback>
     </gazebo>
-    <gazebo reference="wsg_base_mount_right_joint">
-      <implicitSpringDamper>1</implicitSpringDamper>
-      <provideFeedback>true</provideFeedback>
-    </gazebo>
   </xacro:macro>
 </robot>

File: ws/src/ur5_description/robots/wsg.xacro (robot description, xacro)
@@ -1,160 +1,160 @@
 <?xml version="1.0"?>
 <robot xmlns:xacro="http://www.ros.org/wiki/xacro" name="wsg">
-    <xacro:macro name="wsg">
-    <joint name="robot_to_ee" type="fixed">
-        <origin xyz="0.0 -0.1515 0.0" rpy="0.0 0.0 ${pi}" />
-        <parent link="end_middle" />
-        <child link="wsg_base" />
-    </joint>
-    <link name="wsg_base">
-        <visual>
-            <geometry>
-                <mesh filename="package://ur5_description/meshes/collision/wsg50base.stl" />
-            </geometry>
-        </visual>
-        <collision>
-            <geometry>
-                <mesh filename="package://ur5_description/meshes/collision/wsg50base.stl" />
-            </geometry>
-        </collision>
-        <inertial>
-            <mass value="0.7"/>
-            <inertia ixx="0.004433" ixy="0.0" ixz="0.0" iyy="0.00443333156" iyz="0.0" izz="0.0072"/>
-        </inertial>
-    </link>
-    <!-- Right Finger -->
-    <joint name="wsg_base_mount_right_joint" type="prismatic">
-        <origin xyz="0.005 -0.0719 0.0" rpy="0.0 0.0 0.0" />
-        <parent link="wsg_base" />
-        <child link="wsg_finger_mount_right" />
-        <axis xyz="1 0 0" />
-        <limit lower="0" upper="0.050" effort="150.0" velocity="${pi}"/>
-        <dynamics damping="0.4" friction="0.0"/>
-    </joint>
-    <link name="wsg_finger_mount_right">
-        <visual>
-            <geometry>
-                <mesh filename="package://ur5_description/meshes/collision/fingerweiss50_mount.stl" />
-            </geometry>
-        </visual>
-        <collision>
-            <geometry>
-                <mesh filename="package://ur5_description/meshes/collision/fingerweiss50_mount.stl" />
-            </geometry>
-        </collision>
-        <inertial>
-            <mass value="0.5"/>
-            <inertia ixx="0.004433" ixy="0.0" ixz="0.0" iyy="0.00443333156" iyz="0.0" izz="0.0072"/>
-        </inertial>
-    </link>
-    <joint name="wsg_mount_finger_right" type="fixed">
-        <origin xyz="0.0 -0.024 0.0" rpy="${pi} 0.0 0.0" />
-        <parent link="wsg_finger_mount_right" />
-        <child link="wsg_finger_right" />
-    </joint>
-    <link name="wsg_finger_right">
-        <visual>
-            <geometry>
-                <mesh filename="package://ur5_description/meshes/collision/fingerweiss50.stl" />
-            </geometry>
-        </visual>
-        <collision>
-            <geometry>
-                <mesh filename="package://ur5_description/meshes/collision/fingerweiss50.stl" />
-            </geometry>
-        </collision>
-        <inertial>
-            <mass value="0.5"/>
-            <inertia ixx="0.004433" ixy="0.0" ixz="0.0" iyy="0.00443333156" iyz="0.0" izz="0.0072"/>
-        </inertial>
-    </link>
-    <joint name="wsg_fingertip_right" type="fixed">
-        <origin xyz="0.0 -0.072 0.0" rpy="${pi} 0.0 ${pi/2}" />
-        <parent link="wsg_finger_mount_right" />
-        <child link="wsg_fingertip_right" />
-    </joint>
-    <link name="wsg_fingertip_right">
-        <visual>
-            <geometry>
-                <mesh filename="package://ur5_description/meshes/collision/fingerweiss50_tip.stl" />
-            </geometry>
-        </visual>
-        <collision>
-            <geometry>
-                <mesh filename="package://ur5_description/meshes/collision/fingerweiss50_tip.stl" />
-            </geometry>
-        </collision>
-        <inertial>
-            <mass value="0.5"/>
-            <inertia ixx="0.004433" ixy="0.0" ixz="0.0" iyy="0.00443333156" iyz="0.0" izz="0.0072"/>
-        </inertial>
-    </link>
-    <!-- Left Finger -->
-    <joint name="wsg_base_mount_left_joint" type="prismatic">
-        <origin xyz="-0.005 -0.0719 0.0" rpy="0.0 ${pi} 0.0" />
-        <parent link="wsg_base" />
-        <child link="wsg_finger_mount_left" />
-        <axis xyz="1 0 0" />
-        <limit lower="0" upper="0.050" effort="150.0" velocity="${pi}"/>
-        <dynamics damping="0.4" friction="0.0"/>
-    </joint>
-    <link name="wsg_finger_mount_left">
-        <visual>
-            <geometry>
-                <mesh filename="package://ur5_description/meshes/collision/fingerweiss50_mount.stl" />
-            </geometry>
-        </visual>
-        <collision>
-            <geometry>
-                <mesh filename="package://ur5_description/meshes/collision/fingerweiss50_mount.stl" />
-            </geometry>
-        </collision>
-        <inertial>
-            <mass value="0.5"/>
-            <inertia ixx="0.004433" ixy="0.0" ixz="0.0" iyy="0.00443333156" iyz="0.0" izz="0.0072"/>
-        </inertial>
-    </link>
-    <joint name="wsg_mount_finger_left" type="fixed">
-        <origin xyz="0.0 -0.024 0.0" rpy="${pi} 0.0 0.0" />
-        <parent link="wsg_finger_mount_left" />
-        <child link="wsg_finger_left" />
-    </joint>
-    <link name="wsg_finger_left">
-        <visual>
-            <geometry>
-                <mesh filename="package://ur5_description/meshes/collision/fingerweiss50.stl" />
-            </geometry>
-        </visual>
-        <collision>
-            <geometry>
-                <mesh filename="package://ur5_description/meshes/collision/fingerweiss50.stl" />
-            </geometry>
-        </collision>
-        <inertial>
-            <mass value="0.5"/>
-            <inertia ixx="0.004433" ixy="0.0" ixz="0.0" iyy="0.00443333156" iyz="0.0" izz="0.0072"/>
-        </inertial>
-    </link>
-    <joint name="wsg_fingertip_left" type="fixed">
-        <origin xyz="0.0 -0.072 0.0" rpy="${pi} 0.0 ${pi/2}" />
-        <parent link="wsg_finger_mount_left" />
-        <child link="wsg_fingertip_left" />
-    </joint>
-    <link name="wsg_fingertip_left">
-        <visual>
-            <geometry>
-                <mesh filename="package://ur5_description/meshes/collision/fingerweiss50_tip.stl" />
-            </geometry>
-        </visual>
-        <collision>
-            <geometry>
-                <mesh filename="package://ur5_description/meshes/collision/fingerweiss50_tip.stl" />
-            </geometry>
-        </collision>
-        <inertial>
-            <mass value="0.5"/>
-            <inertia ixx="0.004433" ixy="0.0" ixz="0.0" iyy="0.00443333156" iyz="0.0" izz="0.0072"/>
-        </inertial>
-    </link>
-    </xacro:macro>
+  <xacro:macro name="wsg">
+  <joint name="robot_to_ee" type="fixed">
+    <origin xyz="0.0 -0.1515 0.0" rpy="0.0 0.0 ${pi}"/>
+    <parent link="end_middle"/>
+    <child link="wsg_base"/>
+  </joint>
+  <link name="wsg_base">
+    <visual>
+      <geometry>
+        <mesh filename="package://ur5_description/meshes/collision/wsg50base.stl"/>
+      </geometry>
+    </visual>
+    <collision>
+      <geometry>
+        <mesh filename="package://ur5_description/meshes/collision/wsg50base.stl"/>
+      </geometry>
+    </collision>
+    <inertial>
+      <mass value="0.7"/>
+      <inertia ixx="0.004433" ixy="0.0" ixz="0.0" iyy="0.00443333156" iyz="0.0" izz="0.0072"/>
+    </inertial>
+  </link>
+  <!-- right finger -->
+  <joint name="wsg_base_mount_right_joint" type="prismatic">
+    <origin xyz="0.005 -0.0719 0.0" rpy="0.0 0.0 0.0"/>
+    <parent link="wsg_base"/>
+    <child link="wsg_finger_mount_right"/>
+    <axis xyz="1 0 0"/>
+    <limit lower="0" upper="0.050" effort="150.0" velocity="${pi}"/>
+    <dynamics damping="0.4" friction="0.0"/>
+  </joint>
+  <link name="wsg_finger_mount_right">
+    <visual>
+      <geometry>
+        <mesh filename="package://ur5_description/meshes/collision/fingerweiss50_mount.stl"/>
+      </geometry>
+    </visual>
+    <collision>
+      <geometry>
+        <mesh filename="package://ur5_description/meshes/collision/fingerweiss50_mount.stl"/>
+      </geometry>
+    </collision>
+    <inertial>
+      <mass value="0.5"/>
+      <inertia ixx="0.004433" ixy="0.0" ixz="0.0" iyy="0.00443333156" iyz="0.0" izz="0.0072"/>
+    </inertial>
+  </link>
+  <joint name="wsg_mount_finger_right" type="fixed">
+    <origin xyz="0.0 -0.024 0.0" rpy="${pi} 0.0 0.0"/>
+    <parent link="wsg_finger_mount_right"/>
+    <child link="wsg_finger_right"/>
+  </joint>
+  <link name="wsg_finger_right">
+    <visual>
+      <geometry>
+        <mesh filename="package://ur5_description/meshes/collision/fingerweiss50.stl"/>
+      </geometry>
+    </visual>
+    <collision>
+      <geometry>
+        <mesh filename="package://ur5_description/meshes/collision/fingerweiss50.stl"/>
+      </geometry>
+    </collision>
+    <inertial>
+      <mass value="0.5"/>
+      <inertia ixx="0.004433" ixy="0.0" ixz="0.0" iyy="0.00443333156" iyz="0.0" izz="0.0072"/>
+    </inertial>
+  </link>
+  <joint name="wsg_fingertip_right" type="fixed">
+    <origin xyz="0.0 -0.072 0.0" rpy="${pi} 0.0 ${pi/2}"/>
+    <parent link="wsg_finger_mount_right"/>
+    <child link="wsg_fingertip_right"/>
+  </joint>
+  <link name="wsg_fingertip_right">
+    <visual>
+      <geometry>
+        <mesh filename="package://ur5_description/meshes/collision/fingerweiss50_tip.stl"/>
+      </geometry>
+    </visual>
+    <collision>
+      <geometry>
+        <mesh filename="package://ur5_description/meshes/collision/fingerweiss50_tip.stl"/>
+      </geometry>
+    </collision>
+    <inertial>
+      <mass value="0.5"/>
+      <inertia ixx="0.004433" ixy="0.0" ixz="0.0" iyy="0.00443333156" iyz="0.0" izz="0.0072"/>
+    </inertial>
+  </link>
+  <!-- left finger -->
+  <joint name="wsg_base_mount_left_joint" type="prismatic">
+    <origin xyz="-0.005 -0.0719 0.0" rpy="0.0 ${pi} 0.0"/>
+    <parent link="wsg_base"/>
+    <child link="wsg_finger_mount_left"/>
+    <axis xyz="1 0 0"/>
+    <limit lower="0" upper="0.050" effort="150.0" velocity="${pi}"/>
+    <dynamics damping="0.4" friction="0.0"/>
+  </joint>
+  <link name="wsg_finger_mount_left">
+    <visual>
+      <geometry>
+        <mesh filename="package://ur5_description/meshes/collision/fingerweiss50_mount.stl"/>
+      </geometry>
+    </visual>
+    <collision>
+      <geometry>
+        <mesh filename="package://ur5_description/meshes/collision/fingerweiss50_mount.stl"/>
+      </geometry>
+    </collision>
+    <inertial>
+      <mass value="0.5"/>
+      <inertia ixx="0.004433" ixy="0.0" ixz="0.0" iyy="0.00443333156" iyz="0.0" izz="0.0072"/>
+    </inertial>
+  </link>
+  <joint name="wsg_mount_finger_left" type="fixed">
+    <origin xyz="0.0 -0.024 0.0" rpy="${pi} 0.0 0.0"/>
+    <parent link="wsg_finger_mount_left"/>
+    <child link="wsg_finger_left"/>
+  </joint>
+  <link name="wsg_finger_left">
+    <visual>
+      <geometry>
+        <mesh filename="package://ur5_description/meshes/collision/fingerweiss50.stl"/>
+      </geometry>
+    </visual>
+    <collision>
+      <geometry>
+        <mesh filename="package://ur5_description/meshes/collision/fingerweiss50.stl"/>
+      </geometry>
+    </collision>
+    <inertial>
+      <mass value="0.5"/>
+      <inertia ixx="0.004433" ixy="0.0" ixz="0.0" iyy="0.00443333156" iyz="0.0" izz="0.0072"/>
+    </inertial>
+  </link>
+  <joint name="wsg_fingertip_left" type="fixed">
+    <origin xyz="0.0 -0.072 0.0" rpy="${pi} 0.0 ${pi/2}"/>
+    <parent link="wsg_finger_mount_left"/>
+    <child link="wsg_fingertip_left"/>
+  </joint>
+  <link name="wsg_fingertip_left">
+    <visual>
+      <geometry>
+        <mesh filename="package://ur5_description/meshes/collision/fingerweiss50_tip.stl"/>
+      </geometry>
+    </visual>
+    <collision>
+      <geometry>
+        <mesh filename="package://ur5_description/meshes/collision/fingerweiss50_tip.stl"/>
+      </geometry>
+    </collision>
+    <inertial>
+      <mass value="0.5"/>
+      <inertia ixx="0.004433" ixy="0.0" ixz="0.0" iyy="0.00443333156" iyz="0.0" izz="0.0072"/>
+    </inertial>
+  </link>
+  </xacro:macro>
 </robot>
