Commit message: fixed UR5 model for ROS noetic

File: ws/src/ur5_description/robots/ur5_arm.xacro (robot description, xacro)
@@ -2,38 +2,38 @@
 <robot xmlns:xacro="http://www.ros.org/wiki/xacro" name="ur5">
   <!-- properties of the UR5 robot -->
-  <property name="base_mass" value="0.1" />
-  <property name="shoulder_mass" value="0.1" />
-  <property name="upper_arm_mass" value="0.1" />
-  <property name="forearm_mass" value="0.1" />
-  <property name="wrist_1_mass" value="0.1" />
-  <property name="wrist_2_mass" value="0.1" />
-  <property name="wrist_3_mass" value="0.1" />
-  <property name="shoulder_cog" value="0.0 0.00193 -0.02561" />
-  <property name="upper_arm_cog" value="0.0 -0.024201 0.2125" />
-  <property name="forearm_cog" value="0.0 0.0265 0.11993" />
-  <property name="wrist_1_cog" value="0.0 0.110949 0.01634" />
-  <property name="wrist_2_cog" value="0.0 0.0018 0.11099" />
-  <property name="wrist_3_cog" value="0.0 0.001159 0.0" />
-  <property name="ur5_d1" value="0.089159" />
-  <property name="ur5_a2" value="-0.42500" />
-  <property name="ur5_a3" value="-0.39225" />
-  <property name="ur5_d4" value="0.14215" />
-  <property name="ur5_d5" value="0.1" />
-  <property name="ur5_d6" value="0.0983" />
-  <property name="shoulder_offset" value="0.13585" />
-  <property name="elbow_offset" value="-0.1197" />
-  <property name="shoulder_height" value="${ur5_d1}" />
-  <property name="upper_arm_length" value="${-ur5_a2}" />
-  <property name="forearm_length" value="${-ur5_a3}" />
-  <property name="wrist_1_length" value="${ur5_d4 - elbow_offset - shoulder_offset}" />
-  <property name="wrist_2_length" value="${ur5_d5}" />
-  <property name="wrist_3_length" value="${ur5_d6}" />
-  <property name="shoulder_radius" value="0.060" />
-  <property name="upper_arm_radius" value="0.054" />
-  <property name="elbow_radius" value="0.060" />
-  <property name="forearm_radius" value="0.040" />
-  <property name="wrist_radius" value="0.045" />
+  <xacro:property name="base_mass" value="0.1" />
+  <xacro:property name="shoulder_mass" value="0.1" />
+  <xacro:property name="upper_arm_mass" value="0.1" />
+  <xacro:property name="forearm_mass" value="0.1" />
+  <xacro:property name="wrist_1_mass" value="0.1" />
+  <xacro:property name="wrist_2_mass" value="0.1" />
+  <xacro:property name="wrist_3_mass" value="0.1" />
+  <xacro:property name="shoulder_cog" value="0.0 0.00193 -0.02561" />
+  <xacro:property name="upper_arm_cog" value="0.0 -0.024201 0.2125" />
+  <xacro:property name="forearm_cog" value="0.0 0.0265 0.11993" />
+  <xacro:property name="wrist_1_cog" value="0.0 0.110949 0.01634" />
+  <xacro:property name="wrist_2_cog" value="0.0 0.0018 0.11099" />
+  <xacro:property name="wrist_3_cog" value="0.0 0.001159 0.0" />
+  <xacro:property name="ur5_d1" value="0.089159" />
+  <xacro:property name="ur5_a2" value="-0.42500" />
+  <xacro:property name="ur5_a3" value="-0.39225" />
+  <xacro:property name="ur5_d4" value="0.14215" />
+  <xacro:property name="ur5_d5" value="0.1" />
+  <xacro:property name="ur5_d6" value="0.0983" />
+  <xacro:property name="shoulder_offset" value="0.13585" />
+  <xacro:property name="elbow_offset" value="-0.1197" />
+  <xacro:property name="shoulder_height" value="${ur5_d1}" />
+  <xacro:property name="upper_arm_length" value="${-ur5_a2}" />
+  <xacro:property name="forearm_length" value="${-ur5_a3}" />
+  <xacro:property name="wrist_1_length" value="${ur5_d4 - elbow_offset - shoulder_offset}" />
+  <xacro:property name="wrist_2_length" value="${ur5_d5}" />
+  <xacro:property name="wrist_3_length" value="${ur5_d6}" />
+  <xacro:property name="shoulder_radius" value="0.060" />
+  <xacro:property name="upper_arm_radius" value="0.054" />
+  <xacro:property name="elbow_radius" value="0.060" />
+  <xacro:property name="forearm_radius" value="0.040" />
+  <xacro:property name="wrist_radius" value="0.045" />
   <!-- cyldenrical inertia for approximation for the link inertias -->
-  <macro name="cylinder_inertial" params="radius length mass *origin">
+  <!-- <xacro:macro name="cylinder_inertial" params="radius length mass *origin">
     <inertial>
       <mass value="${mass}" />
@@ -41,7 +41,7 @@
       <inertia ixx="${0.0833333 * mass * (3 * radius * radius + length * length)}" ixy="0.0" ixz="0.0" iyy="${0.0833333 * mass * (3 * radius * radius + length * length)}" iyz="0.0" izz="${0.5 * mass * radius * radius}" />
     </inertial>
-  </macro>
+  </xacro:macro> -->
   <!-- the ur5_arm element -->
-  <macro name="ur5_arm">
+  <xacro:macro name="ur5_arm">
     <!-- fix the robot to the Gazebo world coordinate system -->
     <link name="world" />
@@ -50,4 +50,5 @@
       <child link="ur5_link0" />
       <origin xyz="0.0 0.0 0.0" rpy="0.0 0.0 0.0" />
+	  <dynamics damping="1.0"/>
     </joint>
     <!-- link 0 -->
@@ -100,12 +101,12 @@
         </geometry>
       </collision>
-      <cylinder_inertial radius="0.06" length="0.15" mass="${shoulder_mass}">
-        <origin xyz="0.0 0.0 0.0" rpy="0 0 0" />
-      </cylinder_inertial>
-      <!-- <inertial>
+      <!-- <cylinder_inertial radius="0.06" length="0.15" mass="${shoulder_mass}">
+        <origin xyz="0.0 0.0 0.0" rpy="0 0 0" />
+      </cylinder_inertial> -->
+      <inertial>
         <mass value="3.7"/>
         <inertia ixx="0.010267495893" ixy="0.0" ixz="0.0" iyy="0.010267495893" iyz="0.0" izz="0.00666"/>
         <origin rpy="0.0 0.0 0.0" xyz="0.0 0.00193 -0.02561"/>
-      </inertial> -->
+      </inertial>
     </link>
     <!-- joint2 connects link1 and link2 -->
@@ -134,12 +135,12 @@
         </geometry>
       </collision>
-      <cylinder_inertial radius="0.06" length="0.56" mass="${upper_arm_mass}">
+      <!-- <cylinder_inertial radius="0.06" length="0.56" mass="${upper_arm_mass}">
         <origin xyz="0.0 0.0 0.28" rpy="0 0 0" />
-      </cylinder_inertial>
-      <!-- <inertial>
+      </cylinder_inertial> -->
+      <inertial>
         <mass value="8.393"/>
         <inertia ixx="0.22689067591036" ixy="0.0" ixz="0.0" iyy="0.22689067591036" iyz="0.0" izz="0.0151074" />
         <origin rpy="0.0 0.0 0.0" xyz="0.0 -0.024201 0.2125"/>
-      </inertial> -->
+      </inertial>
     </link>
     <!-- joint3 connects link2 and link3 -->
@@ -168,12 +169,12 @@
         </geometry>
       </collision>
-      <cylinder_inertial radius="0.06" length="0.5" mass="${forearm_mass}">
+      <!-- <cylinder_inertial radius="0.06" length="0.5" mass="${forearm_mass}">
         <origin xyz="0.0 0.0 0.25" rpy="0 0 0" />
-      </cylinder_inertial>
-      <!-- <inertial>
+      </cylinder_inertial> -->
+      <inertial>
         <mass value="2.275"/>
         <origin rpy="0.0 0.0 0.0" xyz="0.0 0.0265 0.11993"/>
         <inertia ixx="0.049443313556" ixy="0.0" ixz="0.0" iyy="0.049443313556" iyz="0.0" izz="0.004095" />
-      </inertial> -->
+      </inertial>
     </link>
     <!-- joint4 connects link3 and link4 -->
@@ -201,12 +202,12 @@
         </geometry>
       </collision>
-      <cylinder_inertial radius="0.6" length="0.12" mass="${wrist_1_mass}">
-        <origin xyz="0.0 0.0 0.0" rpy="0 0 0" />
-      </cylinder_inertial>
-      <!-- <inertial>
+      <!-- <cylinder_inertial radius="0.6" length="0.12" mass="${wrist_1_mass}">
+        <origin xyz="0.0 0.0 0.0" rpy="0 0 0" />
+      </cylinder_inertial> -->
+      <inertial>
         <mass value="1.219"/>
         <origin rpy="0.0 0.0 0.0" xyz="0.0 0.110949 0.01634"/>
         <inertia ixx="0.11117275553088" ixy="0.0" ixz="0.0" iyy="0.11117275553088" iyz="0.0" izz="0.21942" />
-      </inertial> -->
+      </inertial>
     </link>
     <!-- joint5 connects link4 and link5 -->
@@ -234,12 +235,12 @@
         </geometry>
       </collision>
-      <cylinder_inertial radius="0.6" length="0.12" mass="${wrist_2_mass}">
-        <origin xyz="0.0 0.0 0.0" rpy="0 0 0" />
-      </cylinder_inertial>
-      <!-- <inertial>
+      <!-- <cylinder_inertial radius="0.6" length="0.12" mass="${wrist_2_mass}">
+        <origin xyz="0.0 0.0 0.0" rpy="0 0 0" />
+      </cylinder_inertial> -->
+      <inertial>
         <mass value="1.219"/>
         <origin rpy="0.0 0.0 0.0" xyz="0.0 0.0018 0.11099"/>
         <inertia ixx="0.11117275553088" ixy="0.0" ixz="0.0" iyy="0.11117275553088" iyz="0.0" izz="0.21942" />
-      </inertial> -->
+      </inertial>
     </link>
     <!-- joint6 connects link5 and link6 -->
@@ -267,13 +268,13 @@
         </geometry>
       </collision>
-      <cylinder_inertial radius="0.6" length="0.12" mass="${wrist_3_mass}">
-        <origin xyz="0.0 0.0 0.0" rpy="0 0 0" />
-      </cylinder_inertial>
-      <!-- <inertial>
+      <!-- <cylinder_inertial radius="0.6" length="0.12" mass="${wrist_3_mass}">
+        <origin xyz="0.0 0.0 0.0" rpy="0 0 0" />
+      </cylinder_inertial> -->
+      <inertial>
         <mass value="0.1879"/>
         <origin rpy="0.0 0.0 0.0" xyz="0.0 0.001159 0.0"/>
         <inertia ixx="0.017136473145408" ixy="0.0" ixz="0.0" iyy="0.017136473145408" iyz="0.0" izz="0.033822" />
-      </inertial> -->
-    </link>
-  </macro>
+      </inertial>
+    </link>
+  </xacro:macro>
 </robot>

Commit message: added xacro file for wsg

File: ws/src/ur5_description/robots/ur5_arm.xacro (robot description, xacro)
@@ -288,5 +288,6 @@
       </inertial>
     </link>
-    <!-- <joint name="ee_fixed_joint" type="fixed">
+    <!--
+      <joint name="ee_fixed_joint" type="fixed">
       <parent link="$u5_link6" />
       <child link = "ee_link" />

Commit message: removed the ur5e robot, added ur5, changed urdf, updated dynamics with jac

File: ws/src/ur5_description/robots/ur5_arm.xacro (robot description, xacro)
@@ -18,7 +18,7 @@
   <xacro:property name="ur5_a2" value="-0.42500"/>
   <xacro:property name="ur5_a3" value="-0.39225"/>
-  <xacro:property name="ur5_d4" value="0.14215"/>
-  <xacro:property name="ur5_d5" value="0.1"/>
-  <xacro:property name="ur5_d6" value="0.0983"/>
+  <xacro:property name="ur5_d4" value="0.10915"/>
+  <xacro:property name="ur5_d5" value="0.09465"/>
+  <xacro:property name="ur5_d6" value="0.0823"/>
   <xacro:property name="shoulder_offset" value="0.13585"/>
   <xacro:property name="elbow_offset" value="-0.1197"/>
@@ -61,14 +61,15 @@
     <link name="ur5_link0">
       <visual>
-        <geometry>
-          <mesh filename="package://ur5_description/meshes/visual/link0.dae"/>
-        </geometry>
-        <material name="LightGrey">
-          <color rgba="0.7 0.7 0.7 1.0"/>
-        </material>
-      </visual>
-      <collision>
-        <geometry>
-          <mesh filename="package://ur5_description/meshes/collision/link0.stl"/>
+        <origin xyz="0.0 0.0 0.003" rpy="0.0 0.0 0.0"/>
+        <geometry>
+          <mesh filename="package://ur5_description/meshes/visual/base.dae"/>
+        </geometry>
+        <material name="LightGrey">
+          <color rgba="0.7 0.7 0.7 1.0"/>
+        </material>
+      </visual>
+      <collision>
+        <geometry>
+          <mesh filename="package://ur5_description/meshes/collision/base.stl"/>
         </geometry>
       </collision>
@@ -97,13 +98,13 @@
       <visual>
         <geometry>
-          <mesh filename="package://ur5_description/meshes/visual/link1.dae"/>
-        </geometry>
-        <material name="LightGrey">
-          <color rgba="0.7 0.7 0.7 1.0"/>
-        </material>
-      </visual>
-      <collision>
-        <geometry>
-          <mesh filename="package://ur5_description/meshes/collision/link1.stl"/>
+          <mesh filename="package://ur5_description/meshes/visual/shoulder.dae"/>
+        </geometry>
+        <material name="LightGrey">
+          <color rgba="0.7 0.7 0.7 1.0"/>
+        </material>
+      </visual>
+      <collision>
+        <geometry>
+          <mesh filename="package://ur5_description/meshes/collision/shoulder.stl"/>
         </geometry>
       </collision>
@@ -132,13 +133,13 @@
       <visual>
         <geometry>
-          <mesh filename="package://ur5_description/meshes/visual/link2.dae"/>
-        </geometry>
-        <material name="LightGrey">
-          <color rgba="0.7 0.7 0.7 1.0"/>
-        </material>
-      </visual>
-      <collision>
-        <geometry>
-          <mesh filename="package://ur5_description/meshes/collision/link2.stl"/>
+          <mesh filename="package://ur5_description/meshes/visual/upperarm.dae"/>
+        </geometry>
+        <material name="LightGrey">
+          <color rgba="0.7 0.7 0.7 1.0"/>
+        </material>
+      </visual>
+      <collision>
+        <geometry>
+          <mesh filename="package://ur5_description/meshes/collision/upperarm.stl"/>
         </geometry>
       </collision>
@@ -167,13 +168,13 @@
       <visual>
         <geometry>
-          <mesh filename="package://ur5_description/meshes/visual/link3.dae"/>
-        </geometry>
-        <material name="LightGrey">
-          <color rgba="0.7 0.7 0.7 1.0"/>
-        </material>
-      </visual>
-      <collision>
-        <geometry>
-          <mesh filename="package://ur5_description/meshes/collision/link3.stl"/>
+          <mesh filename="package://ur5_description/meshes/visual/forearm.dae"/>
+        </geometry>
+        <material name="LightGrey">
+          <color rgba="0.7 0.7 0.7 1.0"/>
+        </material>
+      </visual>
+      <collision>
+        <geometry>
+          <mesh filename="package://ur5_description/meshes/collision/forearm.stl"/>
         </geometry>
       </collision>
@@ -201,13 +202,13 @@
       <visual>
         <geometry>
-          <mesh filename="package://ur5_description/meshes/visual/link4.dae"/>
-        </geometry>
-        <material name="LightGrey">
-          <color rgba="0.7 0.7 0.7 1.0"/>
-        </material>
-      </visual>
-      <collision>
-        <geometry>
-          <mesh filename="package://ur5_description/meshes/collision/link4.stl"/>
+          <mesh filename="package://ur5_description/meshes/visual/wrist1.dae"/>
+        </geometry>
+        <material name="LightGrey">
+          <color rgba="0.7 0.7 0.7 1.0"/>
+        </material>
+      </visual>
+      <collision>
+        <geometry>
+          <mesh filename="package://ur5_description/meshes/collision/wrist1.stl"/>
         </geometry>
       </collision>
@@ -235,13 +236,13 @@
       <visual>
         <geometry>
-          <mesh filename="package://ur5_description/meshes/visual/link5.dae"/>
-        </geometry>
-        <material name="LightGrey">
-          <color rgba="0.7 0.7 0.7 1.0"/>
-        </material>
-      </visual>
-      <collision>
-        <geometry>
-          <mesh filename="package://ur5_description/meshes/collision/link5.stl"/>
+          <mesh filename="package://ur5_description/meshes/visual/wrist2.dae"/>
+        </geometry>
+        <material name="LightGrey">
+          <color rgba="0.7 0.7 0.7 1.0"/>
+        </material>
+      </visual>
+      <collision>
+        <geometry>
+          <mesh filename="package://ur5_description/meshes/collision/wrist2.stl"/>
         </geometry>
       </collision>
@@ -269,18 +270,15 @@
       <visual>
         <geometry>
-          <mesh filename="package://ur5_description/meshes/visual/link6.dae"/>
-        </geometry>
-        <material name="LightGrey">
-          <color rgba="0.7 0.7 0.7 1.0"/>
-        </material>
-      </visual>
-      <collision>
-        <geometry>
-          <mesh filename="package://ur5_description/meshes/collision/link6.stl"/>
-        </geometry>
-      </collision>
-      <!-- <cylinder_inertial radius="0.6" length="0.12" mass="${wrist_3_mass}">
-        <origin xyz="0.0 0.0 0.0" rpy="0 0 0"/>
-      </cylinder_inertial> -->
+          <mesh filename="package://ur5_description/meshes/visual/wrist3.dae"/>
+        </geometry>
+        <material name="LightGrey">
+          <color rgba="0.7 0.7 0.7 1.0"/>
+        </material>
+      </visual>
+      <collision>
+        <geometry>
+          <mesh filename="package://ur5_description/meshes/collision/wrist3.stl"/>
+        </geometry>
+      </collision>
       <inertial>
         <mass value="0.1879"/>
@@ -289,7 +287,14 @@
       </inertial>
     </link>
+    <joint name="ur5_ee_joint" type="fixed">
+        <origin xyz="0.0 0.0823 0.0" rpy="0.0 0.0 0.0"/>
+        <parent link="ur5_link6"/>
+        <child link="ur5_ee"/>
+    </joint>
+    <link name="ur5_ee">
+    </link>
     <joint name="robot_to_ee_end" type="fixed">
-        <origin xyz="0.0 0.25 0.0" rpy="0.0 0.0 0.0"/>
-        <parent link="ur5_link6"/>
+        <origin xyz="0.0 0.1507 0.0" rpy="0.0 0.0 0.0"/>
+        <parent link="ur5_ee"/>
         <child link="ee_tcp"/>
     </joint>

Commit message: added controller

File: ws/src/ur5_description/robots/ur5_arm.xacro (robot description, xacro)
@@ -91,5 +91,5 @@
       <!-- <limit lower="-3.14" upper="3.14" effort="112.0" velocity="3.15"/> -->
       <limit lower="${-pi}" upper="${pi}" effort="112.0" velocity="${pi}"/>
-      <dynamics damping="0.4" friction="0.0"/>
+      <dynamics damping="2" friction="0.0"/>
     </joint>
     <!-- link 1 -->
@@ -126,5 +126,5 @@
       <!-- <limit lower="-3.14" upper="3.14" effort="112.0" velocity="3.15"/> -->
       <limit lower="${-pi}" upper="${pi}" effort="112.0" velocity="${pi}"/>
-      <dynamics damping="0.4" friction="0.0"/>
+      <dynamics damping="2" friction="0.0"/>
     </joint>
     <!-- link 2 -->
@@ -161,5 +161,5 @@
       <!-- <limit lower="-3.14" upper="3.14" effort="112.0" velocity="3.15"/> -->
       <limit lower="${-pi}" upper="${pi}" effort="112.0" velocity="${pi}"/>
-    <dynamics damping="0.4" friction="0.0"/>
+    <dynamics damping="2" friction="0.0"/>
     </joint>
     <!-- link 3 -->

Commit message: added alot

File: ws/src/ur5_description/robots/ur5_arm.xacro (robot description, xacro)
@@ -195,5 +195,5 @@
       <axis xyz="0 1 0"/>
       <!-- <limit lower="-3.14" upper="3.14" effort="28.0" velocity="3.2"/> -->
-      <limit lower="${-1.0 * pi}" upper="${0.25 * pi}" effort="28.0" velocity="${pi}"/>
+      <limit lower="${-pi}" upper="${pi}" effort="28.0" velocity="${pi}"/>
       <dynamics damping="0.3" friction="0.0"/>
     </joint>
