Commit message: added new config for mvoeit

File: ws/src/ur5_description/robots/wsg.xacro (robot description, xacro)
@@ -98,4 +98,5 @@
     <limit lower="0" upper="0.050" effort="150.0" velocity="${pi}"/>
     <dynamics damping="0.4" friction="0.0"/>
+    <mimic joint="wsg_base_mount_right_joint" multiplier="1" offset="0"/>
   </joint>
   <link name="wsg_finger_mount_left">

Commit message: add some color to gripper

File: ws/src/ur5_description/robots/wsg.xacro (robot description, xacro)
@@ -12,4 +12,7 @@
         <mesh filename="package://ur5_description/meshes/collision/wsg50base.stl"/>
       </geometry>
+      <material name="orange">
+        <color rgba="${255/255} ${108/255} ${10/255} 1.0"/>
+      </material>
     </visual>
     <collision>
