Commit message: fixed UR5 for position control

File: ws/src/ur5_description/robots/ur5.gazebo.xacro (robot description, xacro)
@@ -4,4 +4,5 @@
 <!-- link 0 -->
     <gazebo reference="ur5_link0">
+      <static>true</static>
       <selfCollide>true</selfCollide>
       <mu1>0.2</mu1>
@@ -12,4 +13,5 @@
     <!-- link/joint 1 -->
     <gazebo reference="ur5_link1">
+      <static>true</static>
       <selfCollide>true</selfCollide>
       <mu1>0.2</mu1>
@@ -23,4 +25,5 @@
     <!-- link/joint 2 -->
     <gazebo reference="ur5_link2">
+      <static>true</static>
       <selfCollide>true</selfCollide>
       <mu1>0.2</mu1>
@@ -34,4 +37,5 @@
     <!-- link/joint 3 -->
     <gazebo reference="ur5_link3">
+      <static>true</static>
       <selfCollide>true</selfCollide>
       <mu1>0.2</mu1>
@@ -45,4 +49,5 @@
     <!-- link/joint 4 -->
     <gazebo reference="ur5_link4">
+      <static>true</static>
       <selfCollide>true</selfCollide>
       <mu1>0.2</mu1>
@@ -56,4 +61,5 @@
     <!-- link/joint 5 -->
     <gazebo reference="ur5_link5">
+      <static>true</static>
       <selfCollide>true</selfCollide>
       <mu1>0.2</mu1>
@@ -67,4 +73,5 @@
     <!-- link/joint 6 -->
     <gazebo reference="ur5_link6">
+      <static>true</static>
       <selfCollide>true</selfCollide>
       <mu1>0.2</mu1>

File: ws/src/ur5_description/robots/ur5.urdf (robot description, URDF)
Before this commit: robot ur5, 8 links, 7 joints
Links:
- link ur5_link1: mass None -> 3.7
- link ur5_link2: mass None -> 8.393
- link ur5_link3: mass None -> 2.275
- link ur5_link4: mass None -> 1.219
- link ur5_link5: mass None -> 1.219
- link ur5_link6: mass None -> 0.1879
Joints:
- joint ur5_joint1: limit lower=-3.14 upper=3.14 effort=150.0 velocity=3.15 -> lower=-3.141592653589793 upper=3.141592653589793 effort=150.0 velocity=3.141592653589793
- joint ur5_joint2: limit lower=-3.14 upper=3.14 effort=150.0 velocity=3.15 -> lower=-3.141592653589793 upper=3.141592653589793 effort=150.0 velocity=3.141592653589793
- joint ur5_joint3: limit lower=-3.14 upper=3.14 effort=150.0 velocity=3.15 -> lower=-3.141592653589793 upper=3.141592653589793 effort=150.0 velocity=3.141592653589793
- joint ur5_joint4: limit lower=-3.14 upper=3.14 effort=28.0 velocity=3.2 -> lower=-3.141592653589793 upper=0.7853981633974483 effort=28.0 velocity=3.141592653589793
- joint ur5_joint5: limit lower=-3.14 upper=3.14 effort=28.0 velocity=3.2 -> lower=-3.141592653589793 upper=3.141592653589793 effort=28.0 velocity=3.141592653589793
- joint ur5_joint6: limit lower=-3.14 upper=3.14 effort=28.0 velocity=3.2 -> lower=-3.141592653589793 upper=3.141592653589793 effort=28.0 velocity=3.141592653589793

File: ws/src/ur5_description/robots/ur5_arm.xacro (robot description, xacro)
@@ -37,5 +37,5 @@
   <!-- <xacro:macro name="cylinder_inertial" params="radius length mass *origin">
     <inertial>
-      <mass value="${mass}" />
+      <mass value="${0.01 />
       <insert_block name="origin" />
       <inertia ixx="${0.0833333 * mass * (3 * radius * radius + length * length)}" ixy="0.0" ixz="0.0" iyy="${0.0833333 * mass * (3 * radius * radius + length * length)}" iyz="0.0" izz="${0.5 * mass * radius * radius}" />
@@ -43,12 +43,17 @@
   </xacro:macro> -->
   <!-- the ur5_arm element -->
-  <xacro:macro name="ur5_arm">
+  <xacro:macro name="ur5_arm" params="shoulder_pan_lower_limit:=${-pi} shoulder_pan_upper_limit:=${pi}
+    shoulder_lift_lower_limit:=${-pi} shoulder_lift_upper_limit:=${pi}
+    elbow_joint_lower_limit:=${-pi}   elbow_joint_upper_limit:=${pi}
+    wrist_1_lower_limit:=${-pi}       wrist_1_upper_limit:=${pi}
+    wrist_2_lower_limit:=${-pi}       wrist_2_upper_limit:=${pi}
+    wrist_3_lower_limit:=${-pi}       wrist_3_upper_limit:=${pi}
+    safety_pos_margin:=0.15           safety_k_position:=20">
     <!-- fix the robot to the Gazebo world coordinate system -->
     <link name="world" />
     <joint name="robot_to_world" type="fixed">
+      <origin xyz="0.0 0.0 0.0" rpy="0.0 0.0 0.0" />
       <parent link="world" />
       <child link="ur5_link0" />
-      <origin xyz="0.0 0.0 0.0" rpy="0.0 0.0 0.0" />
-	  <dynamics damping="1.0"/>
     </joint>
     <!-- link 0 -->
@@ -72,5 +77,5 @@
       </cylinder_inertial> -->
       <inertial>
-        <mass value="4.0"/>
+        <mass value="0.01"/>
         <inertia ixx="0.004433" ixy="0.0" ixz="0.0" iyy="0.00443333156" iyz="0.0" izz="0.0072"/>
       </inertial>
@@ -82,6 +87,7 @@
       <origin xyz="0.0 0.0 ${shoulder_height}" rpy="0.0 0.0 0.0" />
       <axis xyz="0 0 1" />
-      <limit lower="-3.14" upper="3.14" effort="150.0" velocity="3.15" />
-      <dynamics damping="1.0" />
+      <!-- <limit lower="-3.14" upper="3.14" effort="150.0" velocity="3.15" /> -->
+      <limit lower="${-pi}" upper="${pi}" effort="150.0" velocity="${pi}"/>
+      <dynamics damping="0.4" friction="0.0"/>
     </joint>
     <!-- link 1 -->
@@ -105,5 +111,5 @@
       </cylinder_inertial> -->
       <inertial>
-        <mass value="3.7"/>
+        <mass value="0.01"/>
         <inertia ixx="0.010267495893" ixy="0.0" ixz="0.0" iyy="0.010267495893" iyz="0.0" izz="0.00666"/>
         <origin rpy="0.0 0.0 0.0" xyz="0.0 0.00193 -0.02561"/>
@@ -116,6 +122,7 @@
       <origin xyz="0.0 ${shoulder_offset} 0.0" rpy="0.0 ${pi / 2.0} 0.0" />
       <axis xyz="0 1 0" />
-      <limit lower="-3.14" upper="3.14" effort="150.0" velocity="3.15" />
-      <dynamics damping="1.0" />
+      <!-- <limit lower="-3.14" upper="3.14" effort="150.0" velocity="3.15" /> -->
+      <limit lower="${-pi}" upper="${pi}" effort="150.0" velocity="${pi}"/>
+      <dynamics damping="0.4" friction="0.0"/>
     </joint>
     <!-- link 2 -->
@@ -139,5 +146,5 @@
       </cylinder_inertial> -->
       <inertial>
-        <mass value="8.393"/>
+        <mass value="0.01"/>
         <inertia ixx="0.22689067591036" ixy="0.0" ixz="0.0" iyy="0.22689067591036" iyz="0.0" izz="0.0151074" />
         <origin rpy="0.0 0.0 0.0" xyz="0.0 -0.024201 0.2125"/>
@@ -150,6 +157,7 @@
       <origin xyz="0.0 ${elbow_offset} ${upper_arm_length}" rpy="0.0 0.0 0.0" />
       <axis xyz="0 1 0" />
-      <limit lower="-3.14" upper="3.14" effort="150.0" velocity="3.15" />
-      <dynamics damping="1.0" />
+      <!-- <limit lower="-3.14" upper="3.14" effort="150.0" velocity="3.15" /> -->
+      <limit lower="${-pi}" upper="${pi}" effort="150.0" velocity="${pi}" />
+	  <dynamics damping="0.4" friction="0.0" />
     </joint>
     <!-- link 3 -->
@@ -173,5 +181,5 @@
       </cylinder_inertial> -->
       <inertial>
-        <mass value="2.275"/>
+        <mass value="0.01"/>
         <origin rpy="0.0 0.0 0.0" xyz="0.0 0.0265 0.11993"/>
         <inertia ixx="0.049443313556" ixy="0.0" ixz="0.0" iyy="0.049443313556" iyz="0.0" izz="0.004095" />
@@ -184,6 +192,7 @@
       <origin xyz="0.0 0.0 ${forearm_length}" rpy="0.0 ${pi / 2.0} 0.0" />
       <axis xyz="0 1 0" />
-      <limit lower="-3.14" upper="3.14" effort="28.0" velocity="3.2" />
-      <dynamics damping="1.0" />
+      <!-- <limit lower="-3.14" upper="3.14" effort="28.0" velocity="3.2" /> -->
+      <limit lower="${-1.0 * pi}" upper="${0.25 * pi}" effort="28.0" velocity="${pi}"/>
+      <dynamics damping="0.3" friction="0.0"/>
     </joint>
     <!-- link 4 -->
@@ -206,5 +215,5 @@
       </cylinder_inertial> -->
       <inertial>
-        <mass value="1.219"/>
+        <mass value="0.01"/>
         <origin rpy="0.0 0.0 0.0" xyz="0.0 0.110949 0.01634"/>
         <inertia ixx="0.11117275553088" ixy="0.0" ixz="0.0" iyy="0.11117275553088" iyz="0.0" izz="0.21942" />
@@ -217,6 +226,7 @@
       <origin xyz="0.0 ${wrist_1_length} 0.0" rpy="0.0 0.0 0.0" />
       <axis xyz="0 0 1" />
-      <limit lower="-3.14" upper="3.14" effort="28.0" velocity="3.2" />
-      <dynamics damping="1.0" />
+      <!-- <limit lower="-3.14" upper="3.14" effort="28.0" velocity="3.2" /> -->
+      <limit lower="${-1.0 * pi}" upper="${1.0 * pi}" effort="28.0" velocity="${pi}"/>
+      <dynamics damping="0.3" friction="0.0"/>
     </joint>
     <!-- link 5 -->
@@ -239,5 +249,5 @@
       </cylinder_inertial> -->
       <inertial>
-        <mass value="1.219"/>
+        <mass value="0.01"/>
         <origin rpy="0.0 0.0 0.0" xyz="0.0 0.0018 0.11099"/>
         <inertia ixx="0.11117275553088" ixy="0.0" ixz="0.0" iyy="0.11117275553088" iyz="0.0" izz="0.21942" />
@@ -250,6 +260,7 @@
       <origin xyz="0.0 0.0 ${wrist_2_length}" rpy="0.0 0.0 0.0" />
       <axis xyz="0 1 0" />
-      <limit lower="-3.14" upper="3.14" effort="28.0" velocity="3.2" />
-      <dynamics damping="1.0" />
+      <!-- <limit lower="-3.14" upper="3.14" effort="28.0" velocity="3.2" /> -->
+      <limit lower="${-1.0 * pi}" upper="${1.0 * pi}" effort="28.0" velocity="${pi}"/>
+      <dynamics damping="0.3" friction="0.0"/>
     </joint>
     <!-- link 6 -->
@@ -272,9 +283,15 @@
       </cylinder_inertial> -->
       <inertial>
-        <mass value="0.1879"/>
+        <mass value="0.01"/>
         <origin rpy="0.0 0.0 0.0" xyz="0.0 0.001159 0.0"/>
         <inertia ixx="0.017136473145408" ixy="0.0" ixz="0.0" iyy="0.017136473145408" iyz="0.0" izz="0.033822" />
       </inertial>
     </link>
+    <!-- <joint name="ee_fixed_joint" type="fixed">
+      <parent link="$u5_link6" />
+      <child link = "ee_link" />
+      <origin xyz="0.0 ${wrist_3_length} 0.0" rpy="0.0 0.0 ${pi/2.0}" />
+    </joint>
+	<link name="ee_link" /> -->
   </xacro:macro>
 </robot>

Commit message: added wsg + table + bottle

File: ws/src/ur5_description/robots/ur5.gazebo.xacro (robot description, xacro)
@@ -2,16 +2,14 @@
 <robot xmlns:xacro="http://www.ros.org/wiki/xacro">
   <xacro:macro name="ur5_gazebo">
-<!-- link 0 -->
+  <!-- link 0 -->
     <gazebo reference="ur5_link0">
       <static>true</static>
       <selfCollide>true</selfCollide>
-      <mu1>0.2</mu1>
-      <mu2>0.2</mu2>
-      <static>true</static>
+      <mu1>0.1</mu1>
+      <mu2>0.1</mu2>
       <!-- <material>Gazebo/Grey</material> -->
     </gazebo>
     <!-- link/joint 1 -->
     <gazebo reference="ur5_link1">
-      <static>true</static>
       <selfCollide>true</selfCollide>
       <mu1>0.2</mu1>
@@ -25,5 +23,4 @@
     <!-- link/joint 2 -->
     <gazebo reference="ur5_link2">
-      <static>true</static>
       <selfCollide>true</selfCollide>
       <mu1>0.2</mu1>
@@ -37,5 +34,4 @@
     <!-- link/joint 3 -->
     <gazebo reference="ur5_link3">
-      <static>true</static>
       <selfCollide>true</selfCollide>
       <mu1>0.2</mu1>
@@ -49,5 +45,4 @@
     <!-- link/joint 4 -->
     <gazebo reference="ur5_link4">
-      <static>true</static>
       <selfCollide>true</selfCollide>
       <mu1>0.2</mu1>
@@ -61,5 +56,4 @@
     <!-- link/joint 5 -->
     <gazebo reference="ur5_link5">
-      <static>true</static>
       <selfCollide>true</selfCollide>
       <mu1>0.2</mu1>
@@ -73,5 +67,4 @@
     <!-- link/joint 6 -->
     <gazebo reference="ur5_link6">
-      <static>true</static>
       <selfCollide>true</selfCollide>
       <mu1>0.2</mu1>

File: ws/src/ur5_description/robots/ur5_arm.xacro (robot description, xacro)
@@ -51,7 +51,6 @@
     safety_pos_margin:=0.15           safety_k_position:=20">
     <!-- fix the robot to the Gazebo world coordinate system -->
-    <link name="world" />
-    <joint name="robot_to_world" type="fixed">
-      <origin xyz="0.0 0.0 0.0" rpy="0.0 0.0 0.0" />
+    <joint name="world_to_robot" type="fixed">
+      <origin xyz="0.0 0.0 0.2" rpy="0.0 0.0 0.0" />
       <parent link="world" />
       <child link="ur5_link0" />
@@ -288,11 +287,11 @@
       </inertial>
     </link>
-    <!--
-      <joint name="ee_fixed_joint" type="fixed">
-      <parent link="$u5_link6" />
-      <child link = "ee_link" />
-      <origin xyz="0.0 ${wrist_3_length} 0.0" rpy="0.0 0.0 ${pi/2.0}" />
-    </joint>
-	<link name="ee_link" /> -->
+    <joint name="robot_to_ee_end" type="fixed">
+        <origin xyz="0.0 0.25 0.0" rpy="0.0 0.0 0.0" />
+        <parent link="ur5_link6" />
+        <child link="end_middle" />
+    </joint>
+    <link name="end_middle">
+    </link>
   </xacro:macro>
 </robot>

File: ws/src/ur5_description/robots/ur5_with_wsg.urdf.xacro (robot description, xacro)
@@ -1,4 +1,4 @@
 <?xml version="1.0" encoding="utf-8"?>
-<robot xmlns:xacro="http://www.ros.org/wiki/xacro" name="wsg">
+<robot xmlns:xacro="http://www.ros.org/wiki/xacro" name="ur5">
     <!-- load arm -->
     <xacro:include filename="$(find ur5_description)/robots/ur5_arm.xacro" />
@@ -8,6 +8,7 @@
     <xacro:include filename="$(find ur5_description)/robots/wsg.gazebo.xacro"/>
     <xacro:include filename="$(find ur5_description)/robots/wsg.transmission.xacro" />
-    <xacro:include filename="$(find ur5_description)/robots/wsg.urdf.xacro" />
-    <!-- construct robot -->
+    <xacro:include filename="$(find ur5_description)/robots/wsg.xacro" />
+    <link name="world"/>
+    <!-- construct robot note: make a variable to move the robot -->
     <xacro:ur5_arm />
     <xacro:ur5_gazebo />

File: ws/src/ur5_description/robots/wsg.gazebo.xacro (robot description, xacro)
@@ -4,54 +4,54 @@
     <!-- wsg base -->
     <gazebo reference="wsg_base">
-      <static>true</static>
       <selfCollide>true</selfCollide>
-      <mu1>0.2</mu1>
-      <mu2>0.2</mu2>
-      <static>true</static>
+      <mu1>0.1</mu1>
+      <mu2>0.1</mu2>
       <material>Gazebo/Grey</material>
     </gazebo>
     <!-- Right -->
     <gazebo reference="wsg_finger_mount_right">
-      <static>true</static>
       <selfCollide>true</selfCollide>
-      <mu1>0.2</mu1>
-      <mu2>0.2</mu2>
+      <mu1>0.1</mu1>
+      <mu2>0.1</mu2>
       <material>Gazebo/Grey</material>
     </gazebo>
     <gazebo reference="wsg_finger_right">
-      <static>true</static>
       <selfCollide>true</selfCollide>
-      <mu1>0.2</mu1>
-      <mu2>0.2</mu2>
+      <mu1>0.1</mu1>
+      <mu2>0.1</mu2>
       <material>Gazebo/Black</material>
     </gazebo>
     <gazebo reference="wsg_fingertip_right">
-      <static>true</static>
       <selfCollide>true</selfCollide>
-      <mu1>0.2</mu1>
-      <mu2>0.2</mu2>
+      <mu1>0.1</mu1>
+      <mu2>0.1</mu2>
       <material>Gazebo/Blue</material>
     </gazebo>
     <!-- Left -->
     <gazebo reference="wsg_finger_mount_left">
-      <static>true</static>
       <selfCollide>true</selfCollide>
-      <mu1>0.2</mu1>
-      <mu2>0.2</mu2>
+      <mu1>0.1</mu1>
+      <mu2>0.1</mu2>
       <material>Gazebo/Grey</material>
     </gazebo>
     <gazebo reference="wsg_finger_left">
-      <static>true</static>
       <selfCollide>true</selfCollide>
-      <mu1>0.2</mu1>
-      <mu2>0.2</mu2>
+      <mu1>0.1</mu1>
+      <mu2>0.1</mu2>
       <material>Gazebo/Black</material>
     </gazebo>
     <gazebo reference="wsg_fingertip_left">
-      <static>true</static>
       <selfCollide>true</selfCollide>
-      <mu1>0.2</mu1>
-      <mu2>0.2</mu2>
+      <mu1>0.1</mu1>
+      <mu2>0.1</mu2>
       <material>Gazebo/Blue</material>
+    </gazebo>
+    <gazebo reference="wsg_base_mount_left_joint">
+      <implicitSpringDamper>1</implicitSpringDamper>
+      <provideFeedback>true</provideFeedback>
+    </gazebo>
+    <gazebo reference="wsg_base_mount_right_joint">
+      <implicitSpringDamper>1</implicitSpringDamper>
+      <provideFeedback>true</provideFeedback>
     </gazebo>
   </xacro:macro>

File: ws/src/ur5_description/robots/wsg.transmission.xacro (robot description, xacro)
@@ -6,8 +6,8 @@
       <type>transmission_interface/SimpleTransmission</type>
       <joint name="wsg_base_mount_right_joint">
-        <hardwareInterface>hardware_interface/PositionJointInterface</hardwareInterface>
+        <hardwareInterface>hardware_interface/EffortJointInterface</hardwareInterface>
       </joint>
       <actuator name="wsg_base_mount_right_motor">
-        <hardwareInterface>hardware_interface/PositionJointInterface</hardwareInterface>
+        <hardwareInterface>hardware_interface/EffortJointInterface</hardwareInterface>
         <mechanicalReduction>1</mechanicalReduction>
       </actuator>
@@ -17,8 +17,8 @@
       <type>transmission_interface/SimpleTransmission</type>
       <joint name="wsg_base_mount_left_joint">
-        <hardwareInterface>hardware_interface/PositionJointInterface</hardwareInterface>
+        <hardwareInterface>hardware_interface/EffortJointInterface</hardwareInterface>
       </joint>
       <actuator name="wsg_base_mount_left_motor">
-        <hardwareInterface>hardware_interface/PositionJointInterface</hardwareInterface>
+        <hardwareInterface>hardware_interface/EffortJointInterface</hardwareInterface>
         <mechanicalReduction>1</mechanicalReduction>
       </actuator>

File: ws/src/ur5_description/robots/wsg.xacro (robot description, xacro)
@@ -3,6 +3,6 @@
     <xacro:macro name="wsg">
     <joint name="robot_to_ee" type="fixed">
-        <origin xyz="0.0 0.0985 0.0" rpy="0.0 0.0 ${pi}" />
-        <parent link="ur5_link6" />
+        <origin xyz="0.0 -0.1515 0.0" rpy="0.0 0.0 ${pi}" />
+        <parent link="end_middle" />
         <child link="wsg_base" />
     </joint>
@@ -19,5 +19,5 @@
         </collision>
         <inertial>
-            <mass value="0.01"/>
+            <mass value="0.7"/>
             <inertia ixx="0.004433" ixy="0.0" ixz="0.0" iyy="0.00443333156" iyz="0.0" izz="0.0072"/>
         </inertial>
@@ -44,5 +44,5 @@
         </collision>
         <inertial>
-            <mass value="0.001"/>
+            <mass value="0.5"/>
             <inertia ixx="0.004433" ixy="0.0" ixz="0.0" iyy="0.00443333156" iyz="0.0" izz="0.0072"/>
         </inertial>
@@ -65,5 +65,5 @@
         </collision>
         <inertial>
-            <mass value="0.001"/>
+            <mass value="0.5"/>
             <inertia ixx="0.004433" ixy="0.0" ixz="0.0" iyy="0.00443333156" iyz="0.0" izz="0.0072"/>
         </inertial>
@@ -86,5 +86,5 @@
         </collision>
         <inertial>
-            <mass value="0.001"/>
+            <mass value="0.5"/>
             <inertia ixx="0.004433" ixy="0.0" ixz="0.0" iyy="0.00443333156" iyz="0.0" izz="0.0072"/>
         </inertial>
@@ -111,5 +111,5 @@
         </collision>
         <inertial>
-            <mass value="0.01"/>
+            <mass value="0.5"/>
             <inertia ixx="0.004433" ixy="0.0" ixz="0.0" iyy="0.00443333156" iyz="0.0" izz="0.0072"/>
         </inertial>
@@ -132,5 +132,5 @@
         </collision>
         <inertial>
-            <mass value="0.01"/>
+            <mass value="0.5"/>
             <inertia ixx="0.004433" ixy="0.0" ixz="0.0" iyy="0.00443333156" iyz="0.0" izz="0.0072"/>
         </inertial>
@@ -153,5 +153,5 @@
         </collision>
         <inertial>
-            <mass value="0.001"/>
+            <mass value="0.5"/>
             <inertia ixx="0.004433" ixy="0.0" ixz="0.0" iyy="0.00443333156" iyz="0.0" izz="0.0072"/>
         </inertial>

Commit message: cleanup controllers; workcell moved to rovi_gazebo

File: ws/src/ur5_description/robots/ur5.gazebo.xacro (robot description, xacro)
@@ -5,11 +5,12 @@
     <gazebo reference="ur5_link0">
       <static>true</static>
-      <selfCollide>true</selfCollide>
-      <mu1>0.1</mu1>
-      <mu2>0.1</mu2>
+      <selfCollide>false</selfCollide>
+      <mu1>0.2</mu1>
+      <mu2>0.2</mu2>
       <!-- <material>Gazebo/Grey</material> -->
     </gazebo>
     <!-- link/joint 1 -->
     <gazebo reference="ur5_link1">
+	  <!-- <static>true</static> -->
       <selfCollide>true</selfCollide>
       <mu1>0.2</mu1>

File: ws/src/ur5_description/robots/ur5.urdf.xacro (robot description, xacro)
@@ -1,15 +1,11 @@
 <?xml version="1.0" encoding="utf-8"?>
 <robot xmlns:xacro="http://www.ros.org/wiki/xacro" name="ur5">
-  <!-- load arm + hand -->
-  <xacro:include filename="$(find ur5_description)/robots/ur5_arm.xacro"/>
-  <!-- <xacro:include filename="$(find ur5_description)/robots/ur5_gripper.xacro"/> -->
-  <!-- load gazebo + transmission files -->
-  <xacro:include filename="$(find ur5_description)/robots/ur5.gazebo.xacro"/>
-  <xacro:include filename="$(find ur5_description)/robots/ur5.transmission.xacro"/>
-  <link name="world"/>
-  <!-- construct robot -->
-  <xacro:ur5_arm/>
-  <!-- <xacro:ur5_gripper/> -->
-  <xacro:ur5_gazebo/>
-  <xacro:ur5_transmission/>
+    <!-- load arm -->
+    <xacro:include filename="$(find ur5_description)/robots/ur5_arm.xacro"/>
+    <xacro:include filename="$(find ur5_description)/robots/ur5.gazebo.xacro"/>
+    <xacro:include filename="$(find ur5_description)/robots/ur5.transmission.xacro"/>
+    <!-- construct robot -->
+    <xacro:ur5_arm/>
+    <xacro:ur5_gazebo/>
+    <xacro:ur5_transmission/>
 </robot>

File: ws/src/ur5_description/robots/ur5_arm.xacro (robot description, xacro)
@@ -51,4 +51,5 @@
     safety_pos_margin:=0.15           safety_k_position:=20">
     <!-- fix the robot to the Gazebo world coordinate system -->
+    <link name="world"/>
     <joint name="world_to_robot" type="fixed">
       <origin xyz="0.0 0.0 0.0" rpy="0.0 0.0 0.0"/>
@@ -78,4 +79,5 @@
         <mass value="10.0"/>
         <inertia ixx="0.004433" ixy="0.0" ixz="0.0" iyy="0.00443333156" iyz="0.0" izz="0.0072"/>
+    <origin rpy="0.0 0.0 0.0" xyz="0.0 0.0 0.0"/>
       </inertial>
     </link>
@@ -158,5 +160,5 @@
       <!-- <limit lower="-3.14" upper="3.14" effort="112.0" velocity="3.15"/> -->
       <limit lower="${-pi}" upper="${pi}" effort="112.0" velocity="${pi}"/>
-	  <dynamics damping="0.4" friction="0.0"/>
+    <dynamics damping="0.4" friction="0.0"/>
     </joint>
     <!-- link 3 -->
@@ -290,7 +292,7 @@
         <origin xyz="0.0 0.25 0.0" rpy="0.0 0.0 0.0"/>
         <parent link="ur5_link6"/>
-        <child link="end_middle"/>
-    </joint>
-    <link name="end_middle"/>
+        <child link="ee_tcp"/>
+    </joint>
+    <link name="ee_tcp"/>
   </xacro:macro>
 </robot>

File: ws/src/ur5_description/robots/ur5_with_wsg.urdf.xacro (robot description, xacro)
@@ -9,6 +9,5 @@
     <xacro:include filename="$(find ur5_description)/robots/wsg.transmission.xacro"/>
     <xacro:include filename="$(find ur5_description)/robots/wsg.xacro"/>
-    <link name="world"/>
-    <!-- construct robot note: make a variable to move the robot -->
+    <!-- construct robot -->
     <xacro:ur5_arm/>
     <xacro:ur5_gazebo/>

File: ws/src/ur5_description/robots/wsg.xacro (robot description, xacro)
@@ -2,7 +2,7 @@
 <robot xmlns:xacro="http://www.ros.org/wiki/xacro" name="wsg">
   <xacro:macro name="wsg">
-  <joint name="robot_to_ee" type="fixed">
+  <joint name="gripper_to_ee" type="fixed">
     <origin xyz="0.0 -0.1515 0.0" rpy="0.0 0.0 ${pi}"/>
-    <parent link="end_middle"/>
+    <parent link="ee_tcp"/>
     <child link="wsg_base"/>
   </joint>
