Commit message: fix robot base position (flat with table)

File: ws/src/ur5_description/robots/ur5.gazebo.xacro (robot description, xacro)
@@ -5,5 +5,5 @@
     <gazebo reference="ur5_link0">
       <static>true</static>
-      <selfCollide>false</selfCollide>
+      <selfCollide>true</selfCollide>
       <mu1>0.2</mu1>
       <mu2>0.2</mu2>

File: ws/src/ur5_description/robots/ur5_arm.xacro (robot description, xacro)
@@ -59,4 +59,5 @@
     <!-- link 0 -->
     <!-- base link -->
+    <!-- visual and collision meshes are slighly offset such that the base can he placed on a surface -->
     <link name="ur5_link0">
       <visual>
@@ -70,4 +71,5 @@
       </visual>
       <collision>
+        <origin xyz="0.0 0.0 0.005" rpy="0.0 0.0 0.0"/>
         <geometry>
           <mesh filename="package://ur5_description/meshes/collision/base.stl"/>
