Commit message: improved grasping

File: ws/src/ur5_description/robots/wsg.gazebo.xacro (robot description, xacro)
@@ -2,4 +2,6 @@
 <robot xmlns:xacro="http://www.ros.org/wiki/xacro">
   <xacro:macro name="wsg_gazebo">
+    <!-- friction values -->
+    <!-- https://answers.ros.org/question/302358/anyone-whos-succeeded-with-grasping-using-ros-and-gazebo-what-advice-do-you-have-to-offer/?answer=348927#post-id-348927 -->
     <!-- wsg base -->
     <gazebo reference="wsg_base">
@@ -7,6 +9,27 @@
       <gravity>0</gravity>
       <turnGravityOff>true</turnGravityOff>
-      <mu1>2.0</mu1>
-      <mu2>1.5</mu2>
+      <collision>
+      <surface>
+        <friction>
+          <torsional>
+            <coefficient>10.0</coefficient>
+            <use_patch_radius>true</use_patch_radius>
+            <patch_radius>0.05</patch_radius>
+          </torsional>
+        </friction>
+        <contact>
+          <poissons_ratio>0.5</poissons_ratio>
+          <elastic_modulus>1e8</elastic_modulus>
+        </contact>
+      </surface>
+      </collision>
+      <mu1>10</mu1>
+      <mu2>10</mu2>
+      <maxVel>1</maxVel>
+      <kp>1000000.0</kp>
+      <kd>100.0</kd>
+      <fdir1>0 0 1</fdir1>
+      <minDepth>0.0</minDepth>
+      <maxContacts>100</maxContacts>
       <material>Gazebo/Grey</material>
     </gazebo>
@@ -16,7 +39,28 @@
       <gravity>0</gravity>
       <turnGravityOff>true</turnGravityOff>
-      <mu1>2.0</mu1>
-      <mu2>1.5</mu2>
-      <material>Gazebo/Grey</material>
+      <collision>
+      <surface>
+        <friction>
+          <torsional>
+            <coefficient>10.0</coefficient>
+            <use_patch_radius>true</use_patch_radius>
+            <patch_radius>0.05</patch_radius>
+          </torsional>
+        </friction>
+        <contact>
+          <poissons_ratio>0.5</poissons_ratio>
+          <elastic_modulus>1e8</elastic_modulus>
+        </contact>
+      </surface>
+      </collision>
+      <mu1>10</mu1>
+      <mu2>10</mu2>
+      <maxVel>1</maxVel>
+      <kp>1000000.0</kp>
+      <kd>100.0</kd>
+      <fdir1>0 0 1</fdir1>
+      <minDepth>0.0</minDepth>
+      <maxContacts>100</maxContacts>
+        <material>Gazebo/Grey</material>
     </gazebo>
     <gazebo reference="wsg_finger_right">
@@ -24,7 +68,28 @@
       <gravity>0</gravity>
       <turnGravityOff>true</turnGravityOff>
-      <mu1>2.0</mu1>
-      <mu2>1.5</mu2>
-      <material>Gazebo/Black</material>
+      <collision>
+      <surface>
+        <friction>
+          <torsional>
+            <coefficient>10.0</coefficient>
+            <use_patch_radius>true</use_patch_radius>
+            <patch_radius>0.05</patch_radius>
+          </torsional>
+        </friction>
+        <contact>
+          <poissons_ratio>0.5</poissons_ratio>
+          <elastic_modulus>1e8</elastic_modulus>
+        </contact>
+      </surface>
+      </collision>
+      <mu1>10</mu1>
+      <mu2>10</mu2>
+      <maxVel>1</maxVel>
+      <kp>1000000.0</kp>
+      <kd>100.0</kd>
+      <fdir1>0 0 1</fdir1>
+      <minDepth>0.0</minDepth>
+      <maxContacts>100</maxContacts>
+        <material>Gazebo/Black</material>
     </gazebo>
     <gazebo reference="wsg_fingertip_right">
@@ -32,7 +97,28 @@
       <gravity>0</gravity>
       <turnGravityOff>true</turnGravityOff>
-      <mu1>2.0</mu1>
-      <mu2>1.5</mu2>
-      <material>Gazebo/Blue</material>
+      <collision>
+      <surface>
+        <friction>
+          <torsional>
+            <coefficient>10.0</coefficient>
+            <use_patch_radius>true</use_patch_radius>
+            <patch_radius>0.05</patch_radius>
+          </torsional>
+        </friction>
+        <contact>
+          <poissons_ratio>0.5</poissons_ratio>
+          <elastic_modulus>1e8</elastic_modulus>
+        </contact>
+      </surface>
+      </collision>
+      <mu1>10</mu1>
+      <mu2>10</mu2>
+      <maxVel>1</maxVel>
+      <kp>1000000.0</kp>
+      <kd>100.0</kd>
+      <fdir1>0 0 1</fdir1>
+      <minDepth>0.0</minDepth>
+      <maxContacts>100</maxContacts>
+      <material>Gazebo/RedBright</material>
     </gazebo>
     <gazebo reference="wsg_base_mount_right_joint">
@@ -45,7 +131,28 @@
       <gravity>0</gravity>
       <turnGravityOff>true</turnGravityOff>
-      <mu1>2.0</mu1>
-      <mu2>1.5</mu2>
-      <material>Gazebo/Grey</material>
+      <collision>
+      <surface>
+        <friction>
+          <torsional>
+            <coefficient>10.0</coefficient>
+            <use_patch_radius>true</use_patch_radius>
+            <patch_radius>0.05</patch_radius>
+          </torsional>
+        </friction>
+        <contact>
+          <poissons_ratio>0.5</poissons_ratio>
+          <elastic_modulus>1e8</elastic_modulus>
+        </contact>
+      </surface>
+      </collision>
+      <mu1>10</mu1>
+      <mu2>10</mu2>
+      <maxVel>1</maxVel>
+      <kp>1000000.0</kp>
+      <kd>100.0</kd>
+      <fdir1>0 0 1</fdir1>
+      <minDepth>0.0</minDepth>
+      <maxContacts>100</maxContacts>
+        <material>Gazebo/Grey</material>
     </gazebo>
     <gazebo reference="wsg_finger_left">
@@ -53,6 +160,27 @@
       <gravity>0</gravity>
       <turnGravityOff>true</turnGravityOff>
-      <mu1>2.0</mu1>
-      <mu2>1.5</mu2>
+      <collision>
+      <surface>
+        <friction>
+          <torsional>
+            <coefficient>10.0</coefficient>
+            <use_patch_radius>true</use_patch_radius>
+            <patch_radius>0.05</patch_radius>
+          </torsional>
+        </friction>
+        <contact>
+          <poissons_ratio>0.5</poissons_ratio>
+          <elastic_modulus>1e8</elastic_modulus>
+        </contact>
+      </surface>
+      </collision>
+      <mu1>10</mu1>
+      <mu2>10</mu2>
+      <maxVel>1</maxVel>
+      <kp>1000000.0</kp>
+      <kd>100.0</kd>
+      <fdir1>0 0 1</fdir1>
+      <minDepth>0.0</minDepth>
+      <maxContacts>100</maxContacts>
       <material>Gazebo/Black</material>
     </gazebo>
@@ -61,7 +189,28 @@
       <gravity>0</gravity>
       <turnGravityOff>true</turnGravityOff>
-      <mu1>2.0</mu1>
-      <mu2>1.5</mu2>
-      <material>Gazebo/Blue</material>
+      <collision>
+      <surface>
+        <friction>
+          <torsional>
+            <coefficient>10.0</coefficient>
+            <use_patch_radius>true</use_patch_radius>
+            <patch_radius>0.05</patch_radius>
+          </torsional>
+        </friction>
+        <contact>
+          <poissons_ratio>0.5</poissons_ratio>
+          <elastic_modulus>1e8</elastic_modulus>
+        </contact>
+      </surface>
+      </collision>
+      <mu1>10</mu1>
+      <mu2>10</mu2>
+      <maxVel>1</maxVel>
+      <kp>1000000.0</kp>
+      <kd>100.0</kd>
+      <fdir1>0 0 1</fdir1>
+      <minDepth>0.0</minDepth>
+      <maxContacts>100</maxContacts>
+      <material>Gazebo/RedBright</material>
     </gazebo>
     <gazebo reference="wsg_base_mount_left_joint">
