Commit message: update UR5 robot; needs limits and gripper

File: ws/src/ur5_description/robots/old/ur5.transmission.xacro (robot description, xacro)
@@ -1,13 +1,11 @@
 <?xml version="1.0"?>
-<robot xmlns:xacro="http://www.ros.org/wiki/xacro">
+<robot xmlns:xacro="http://www.ros.org/wiki/xacro" name="ur5_transmission">
   <xacro:macro name="ur5_transmission">
-    <!-- Load Gazebo lib with desired parameters -->
     <gazebo>
-    <plugin name="gazebo_ros_control" filename="libgazebo_ros_control.so" />
+      <plugin name="gazebo_ros_control" filename="libgazebo_ros_control.so" />
     </gazebo>
-    <!-- transmission joint 1 -->
     <transmission name="ur5_tran_1">
       <type>transmission_interface/SimpleTransmission</type>
-      <joint name="ur5_joint1">
+      <joint name="ur5_joint_1">
         <hardwareInterface>hardware_interface/PositionJointInterface</hardwareInterface>
       </joint>
@@ -17,8 +15,7 @@
       </actuator>
     </transmission>
-    <!-- transmission joint 2 -->
     <transmission name="ur5_tran_2">
       <type>transmission_interface/SimpleTransmission</type>
-      <joint name="ur5_joint2">
+      <joint name="ur5_joint_2">
         <hardwareInterface>hardware_interface/PositionJointInterface</hardwareInterface>
       </joint>
@@ -28,8 +25,7 @@
       </actuator>
     </transmission>
-    <!-- transmission joint 3 -->
     <transmission name="ur5_tran_3">
       <type>transmission_interface/SimpleTransmission</type>
-      <joint name="ur5_joint3">
+      <joint name="ur5_joint_3">
         <hardwareInterface>hardware_interface/PositionJointInterface</hardwareInterface>
       </joint>
@@ -39,8 +35,7 @@
       </actuator>
     </transmission>
-    <!-- transmission joint 4 -->
     <transmission name="ur5_tran_4">
       <type>transmission_interface/SimpleTransmission</type>
-      <joint name="ur5_joint4">
+      <joint name="ur5_joint_4">
         <hardwareInterface>hardware_interface/PositionJointInterface</hardwareInterface>
       </joint>
@@ -50,8 +45,7 @@
       </actuator>
     </transmission>
-    <!-- transmission joint 5 -->
     <transmission name="ur5_tran_5">
       <type>transmission_interface/SimpleTransmission</type>
-      <joint name="ur5_joint5">
+      <joint name="ur5_joint_5">
         <hardwareInterface>hardware_interface/PositionJointInterface</hardwareInterface>
       </joint>
@@ -61,8 +55,7 @@
       </actuator>
     </transmission>
-    <!-- transmission joint 6 -->
     <transmission name="ur5_tran_6">
       <type>transmission_interface/SimpleTransmission</type>
-      <joint name="ur5_joint6">
+      <joint name="ur5_joint_6">
         <hardwareInterface>hardware_interface/PositionJointInterface</hardwareInterface>
       </joint>
@@ -72,24 +65,23 @@
       </actuator>
     </transmission>
-    <!-- transmission gripper -->
     <transmission name="wsg_tran_left">
-        <type>transmission_interface/SimpleTransmission</type>
-        <joint name="joint_wsg_gripper_left">
-          <hardwareInterface>hardware_interface/PositionJointInterface</hardwareInterface>
-        </joint>
-        <actuator name="wsg_motor_left">
-          <hardwareInterface>hardware_interface/PositionJointInterface</hardwareInterface>
-          <mechanicalReduction>1</mechanicalReduction>
-        </actuator>
-      </transmission>
-      <transmission name="wsg_tran_right">
-        <type>transmission_interface/SimpleTransmission</type>
-        <joint name="joint_wsg_gripper_right">
-          <hardwareInterface>hardware_interface/PositionJointInterface</hardwareInterface>
-        </joint>
-        <actuator name="wsg_motor_right">
-          <hardwareInterface>hardware_interface/PositionJointInterface</hardwareInterface>
-          <mechanicalReduction>1</mechanicalReduction>
-        </actuator>
+      <type>transmission_interface/SimpleTransmission</type>
+      <joint name="joint_wsg_gripper_left">
+        <hardwareInterface>hardware_interface/PositionJointInterface</hardwareInterface>
+      </joint>
+      <actuator name="wsg_motor_left">
+        <hardwareInterface>hardware_interface/PositionJointInterface</hardwareInterface>
+        <mechanicalReduction>1</mechanicalReduction>
+      </actuator>
+    </transmission>
+    <transmission name="wsg_tran_right">
+      <type>transmission_interface/SimpleTransmission</type>
+      <joint name="joint_wsg_gripper_right">
+        <hardwareInterface>hardware_interface/PositionJointInterface</hardwareInterface>
+      </joint>
+      <actuator name="wsg_motor_right">
+        <hardwareInterface>hardware_interface/PositionJointInterface</hardwareInterface>
+        <mechanicalReduction>1</mechanicalReduction>
+      </actuator>
     </transmission>
   </xacro:macro>

File: ws/src/ur5_description/robots/ur5.gazebo.xacro (robot description, xacro)
@@ -1,76 +1,79 @@
 <?xml version="1.0"?>
 <robot xmlns:xacro="http://www.ros.org/wiki/xacro">
-    <xacro:macro name="ur5_gazebo">
-        <!-- Link0 -->
-        <gazebo reference="ur5_link0">
-            <!-- <selfCollide>true</selfCollide> -->
-            <!-- <turnGravityOff>true</turnGravityOff> -->
-            <!-- <static>true</static> -->
-        </gazebo>
-        <!-- Link1 -->
-        <gazebo reference="ur5_link1">
-            <!-- <selfCollide>true</selfCollide> -->
-            <!-- <turnGravityOff>true</turnGravityOff> -->
-			<mu1>0.2</mu1>
-            <mu2>0.2</mu2>
-        </gazebo>
-        <!-- Link2 -->
-        <gazebo reference="ur5_link2">
-            <!-- <selfCollide>true</selfCollide> -->
-            <!-- <turnGravityOff>true</turnGravityOff> -->
-			<mu1>0.2</mu1>
-            <mu2>0.2</mu2>
-        </gazebo>
-        <!-- Link3 -->
-        <gazebo reference="ur5_link3">
-            <!-- <selfCollide>true</selfCollide> -->
-            <!-- <turnGravityOff>true</turnGravityOff> -->
-			<mu1>0.2</mu1>
-            <mu2>0.2</mu2>
-        </gazebo>
-        <!-- Link4 -->
-        <gazebo reference="ur5_link4">
-            <!-- <selfCollide>true</selfCollide> -->
-            <!-- <turnGravityOff>true</turnGravityOff> -->
-			<mu1>0.2</mu1>
-            <mu2>0.2</mu2>
-        </gazebo>
-        <!-- Link5 -->
-        <gazebo reference="ur5_link5">
-            <!-- <selfCollide>true</selfCollide> -->
-            <!-- <turnGravityOff>true</turnGravityOff> -->
-			<mu1>0.2</mu1>
-            <mu2>0.2</mu2>
-        </gazebo>
-        <!-- Link6 -->
-        <gazebo reference="ur5_link6">
-            <!-- <selfCollide>true</selfCollide> -->
-            <!-- <turnGravityOff>true</turnGravityOff> -->
-			<mu1>0.2</mu1>
-            <mu2>0.2</mu2>
-        </gazebo>
-        <!-- Wsg Base -->
-        <gazebo reference="wsg_base">
-            <material>Gazebo/Grey</material>
-            <!-- <turnGravityOff>true</turnGravityOff> -->
-        </gazebo>
-        <!-- Wsg left -->
-        <gazebo reference="wsg_gripper_left">
-            <material>Gazebo/Grey</material>
-            <!-- <turnGravityOff>true</turnGravityOff> -->
-        </gazebo>
-        <gazebo reference="wsg_finger_left">
-            <material>Gazebo/Blue</material>
-            <!-- <turnGravityOff>true</turnGravityOff> -->
-        </gazebo>
-        <!-- Wsg right -->
-        <gazebo reference="wsg_gripper_right">
-            <material>Gazebo/Grey</material>
-            <!-- <turnGravityOff>true</turnGravityOff> -->
-        </gazebo>
-        <gazebo reference="wsg_finger_right">
-            <material>Gazebo/Blue</material>
-            <!-- <turnGravityOff>true</turnGravityOff> -->
-        </gazebo>
-    </xacro:macro>
+  <xacro:macro name="ur5_gazebo">
+<!-- link 0 -->
+    <gazebo reference="ur5_link0">
+      <selfCollide>true</selfCollide>
+      <mu1>0.2</mu1>
+      <mu2>0.2</mu2>
+      <static>true</static>
+      <!-- <material>Gazebo/Grey</material> -->
+    </gazebo>
+    <!-- link/joint 1 -->
+    <gazebo reference="ur5_link1">
+      <selfCollide>true</selfCollide>
+      <mu1>0.2</mu1>
+      <mu2>0.2</mu2>
+      <!-- <material>Gazebo/White</material> -->
+    </gazebo>
+    <gazebo reference="ur5_joint1">
+      <implicitSpringDamper>1</implicitSpringDamper>
+      <provideFeedback>true</provideFeedback>
+    </gazebo>
+    <!-- link/joint 2 -->
+    <gazebo reference="ur5_link2">
+      <selfCollide>true</selfCollide>
+      <mu1>0.2</mu1>
+      <mu2>0.2</mu2>
+      <!-- <material>Gazebo/White</material> -->
+    </gazebo>
+    <gazebo reference="ur5_joint2">
+      <implicitSpringDamper>1</implicitSpringDamper>
+      <provideFeedback>true</provideFeedback>
+    </gazebo>
+    <!-- link/joint 3 -->
+    <gazebo reference="ur5_link3">
+      <selfCollide>true</selfCollide>
+      <mu1>0.2</mu1>
+      <mu2>0.2</mu2>
+      <!-- <material>Gazebo/White</material> -->
+    </gazebo>
+    <gazebo reference="ur5_joint3">
+      <implicitSpringDamper>1</implicitSpringDamper>
+      <provideFeedback>true</provideFeedback>
+    </gazebo>
+    <!-- link/joint 4 -->
+    <gazebo reference="ur5_link4">
+      <selfCollide>true</selfCollide>
+      <mu1>0.2</mu1>
+      <mu2>0.2</mu2>
+      <!-- <material>Gazebo/White</material> -->
+    </gazebo>
+    <gazebo reference="ur5_joint4">
+      <implicitSpringDamper>1</implicitSpringDamper>
+      <provideFeedback>true</provideFeedback>
+    </gazebo>
+    <!-- link/joint 5 -->
+    <gazebo reference="ur5_link5">
+      <selfCollide>true</selfCollide>
+      <mu1>0.2</mu1>
+      <mu2>0.2</mu2>
+      <!-- <material>Gazebo/White</material> -->
+    </gazebo>
+    <gazebo reference="ur5_joint5">
+      <implicitSpringDamper>1</implicitSpringDamper>
+      <provideFeedback>true</provideFeedback>
+    </gazebo>
+    <!-- link/joint 6 -->
+    <gazebo reference="ur5_link6">
+      <selfCollide>true</selfCollide>
+      <mu1>0.2</mu1>
+      <mu2>0.2</mu2>
+      <!-- <material>Gazebo/White</material> -->
+    </gazebo>
+    <gazebo reference="ur5_joint6">
+      <implicitSpringDamper>1</implicitSpringDamper>
+      <provideFeedback>true</provideFeedback>
+    </gazebo>
+  </xacro:macro>
 </robot>

File: ws/src/ur5_description/robots/ur5.transmission.xacro (robot description, xacro)
@@ -1,84 +1,73 @@
 <?xml version="1.0"?>
-<robot xmlns:xacro="http://www.ros.org/wiki/xacro" name="ur5_transmission">
+<robot xmlns:xacro="http://www.ros.org/wiki/xacro">
   <xacro:macro name="ur5_transmission">
+    <!-- Load Gazebo lib with desired parameters -->
     <gazebo>
-      <plugin name="gazebo_ros_control" filename="libgazebo_ros_control.so" />
-    </gazebo>
-    <transmission name="ur5_tran_1">
+		<plugin name="gazebo_ros_control" filename="libgazebo_ros_control.so">
+			<!-- <robotNamespace>/MYROBOT</robotNamespace> -->
+		</plugin>
+	</gazebo>
+    <!-- transmission joint 1 -->
+    <transmission name="ur5_tran1">
       <type>transmission_interface/SimpleTransmission</type>
-      <joint name="ur5_joint_1">
+      <joint name="ur5_joint1">
         <hardwareInterface>hardware_interface/PositionJointInterface</hardwareInterface>
       </joint>
-      <actuator name="ur5_motor_1">
+      <actuator name="ur5_motor1">
         <hardwareInterface>hardware_interface/PositionJointInterface</hardwareInterface>
         <mechanicalReduction>1</mechanicalReduction>
       </actuator>
     </transmission>
-    <transmission name="ur5_tran_2">
+    <!-- transmission joint 2 -->
+    <transmission name="ur5_tran2">
       <type>transmission_interface/SimpleTransmission</type>
-      <joint name="ur5_joint_2">
+      <joint name="ur5_joint2">
         <hardwareInterface>hardware_interface/PositionJointInterface</hardwareInterface>
       </joint>
-      <actuator name="ur5_motor_2">
+      <actuator name="ur5_motor2">
         <hardwareInterface>hardware_interface/PositionJointInterface</hardwareInterface>
         <mechanicalReduction>1</mechanicalReduction>
       </actuator>
     </transmission>
-    <transmission name="ur5_tran_3">
+    <!-- transmission joint 3 -->
+    <transmission name="ur5_tran3">
       <type>transmission_interface/SimpleTransmission</type>
-      <joint name="ur5_joint_3">
+      <joint name="ur5_joint3">
         <hardwareInterface>hardware_interface/PositionJointInterface</hardwareInterface>
       </joint>
-      <actuator name="ur5_motor_3">
+      <actuator name="ur5_motor3">
         <hardwareInterface>hardware_interface/PositionJointInterface</hardwareInterface>
         <mechanicalReduction>1</mechanicalReduction>
       </actuator>
     </transmission>
-    <transmission name="ur5_tran_4">
+    <!-- transmission joint 4 -->
+    <transmission name="ur5_tran4">
       <type>transmission_interface/SimpleTransmission</type>
-      <joint name="ur5_joint_4">
+      <joint name="ur5_joint4">
         <hardwareInterface>hardware_interface/PositionJointInterface</hardwareInterface>
       </joint>
-      <actuator name="ur5_motor_4">
+      <actuator name="ur5_motor4">
         <hardwareInterface>hardware_interface/PositionJointInterface</hardwareInterface>
         <mechanicalReduction>1</mechanicalReduction>
       </actuator>
     </transmission>
-    <transmission name="ur5_tran_5">
+    <!-- transmission joint 5 -->
+    <transmission name="ur5_tran5">
       <type>transmission_interface/SimpleTransmission</type>
-      <joint name="ur5_joint_5">
+      <joint name="ur5_joint5">
         <hardwareInterface>hardware_interface/PositionJointInterface</hardwareInterface>
       </joint>
-      <actuator name="ur5_motor_5">
+      <actuator name="ur5_motor5">
         <hardwareInterface>hardware_interface/PositionJointInterface</hardwareInterface>
         <mechanicalReduction>1</mechanicalReduction>
       </actuator>
     </transmission>
-    <transmission name="ur5_tran_6">
+    <!-- transmission joint 6 -->
+    <transmission name="ur5_tran6">
       <type>transmission_interface/SimpleTransmission</type>
-      <joint name="ur5_joint_6">
+      <joint name="ur5_joint6">
         <hardwareInterface>hardware_interface/PositionJointInterface</hardwareInterface>
       </joint>
-      <actuator name="ur5_motor_6">
-        <hardwareInterface>hardware_interface/PositionJointInterface</hardwareInterface>
-        <mechanicalReduction>1</mechanicalReduction>
-      </actuator>
-    </transmission>
-    <transmission name="wsg_tran_left">
-      <type>transmission_interface/SimpleTransmission</type>
-      <joint name="joint_wsg_gripper_left">
-        <hardwareInterface>hardware_interface/PositionJointInterface</hardwareInterface>
-      </joint>
-      <actuator name="wsg_motor_left">
-        <hardwareInterface>hardware_interface/PositionJointInterface</hardwareInterface>
-        <mechanicalReduction>1</mechanicalReduction>
-      </actuator>
-    </transmission>
-    <transmission name="wsg_tran_right">
-      <type>transmission_interface/SimpleTransmission</type>
-      <joint name="joint_wsg_gripper_right">
-        <hardwareInterface>hardware_interface/PositionJointInterface</hardwareInterface>
-      </joint>
-      <actuator name="wsg_motor_right">
+      <actuator name="ur5_motor6">
         <hardwareInterface>hardware_interface/PositionJointInterface</hardwareInterface>
         <mechanicalReduction>1</mechanicalReduction>

File: ws/src/ur5_description/robots/ur5.urdf.xacro (robot description, xacro)
@@ -5,8 +5,9 @@
   <!-- <xacro:include filename="$(find ur5_description)/robots/ur5_gripper.xacro" /> -->
   <!-- load gazebo + transmission files -->
-  <xacro:include filename="$(find franka_description)/robots/ur5.gazebo.xacro" />
-  <xacro:include filename="$(find franka_description)/robots/ur5.transmission.xacro" />
+  <xacro:include filename="$(find ur5_description)/robots/ur5.gazebo.xacro" />
+  <xacro:include filename="$(find ur5_description)/robots/ur5.transmission.xacro" />
   <!-- construct robot -->
   <xacro:ur5_arm />
+  <!-- <xacro:ur5_gripper /> -->
   <xacro:ur5_gazebo />
   <xacro:ur5_transmission />
