Commit message: update UR5 robot; needs limits and gripper

File: ws/src/ur5_description/robots/ur5_arm.xacro (robot description, xacro)
@@ -52,4 +52,5 @@
     </joint>
     <!-- link 0 -->
+    <!-- base link -->
     <link name="ur5_link0">
       <visual>
@@ -66,7 +67,11 @@
         </geometry>
       </collision>
-      <cylinder_inertial radius="0.06" length="0.05" mass="${base_mass}">
-        <origin xyz="0.0 0.0 0.0" rpy="0 0 0" />
-      </cylinder_inertial>
+      <!-- <cylinder_inertial radius="0.06" length="0.05" mass="${base_mass}">
+        <origin xyz="0.0 0.0 0.0" rpy="0 0 0" />
+      </cylinder_inertial> -->
+      <inertial>
+        <mass value="4.0"/>
+        <inertia ixx="0.004433" ixy="0.0" ixz="0.0" iyy="0.00443333156" iyz="0.0" izz="0.0072"/>
+      </inertial>
     </link>
     <!-- joint1 connects link0 and link1 -->
@@ -77,7 +82,8 @@
       <axis xyz="0 0 1" />
       <limit lower="-3.14" upper="3.14" effort="150.0" velocity="3.15" />
-      <dynamics damping="1" friction="1" />
+      <dynamics damping="1.0" />
     </joint>
     <!-- link 1 -->
+    <!-- shoulder link -->
     <link name="ur5_link1">
       <visual>
@@ -97,4 +103,9 @@
         <origin xyz="0.0 0.0 0.0" rpy="0 0 0" />
       </cylinder_inertial>
+      <!-- <inertial>
+        <mass value="3.7"/>
+        <inertia ixx="0.010267495893" ixy="0.0" ixz="0.0" iyy="0.010267495893" iyz="0.0" izz="0.00666"/>
+        <origin rpy="0.0 0.0 0.0" xyz="0.0 0.00193 -0.02561"/>
+      </inertial> -->
     </link>
     <!-- joint2 connects link1 and link2 -->
@@ -105,7 +116,8 @@
       <axis xyz="0 1 0" />
       <limit lower="-3.14" upper="3.14" effort="150.0" velocity="3.15" />
-      <dynamics damping="1" friction="1" />
+      <dynamics damping="1.0" />
     </joint>
     <!-- link 2 -->
+    <!-- upper arm link -->
     <link name="ur5_link2">
       <visual>
@@ -125,4 +137,9 @@
         <origin xyz="0.0 0.0 0.28" rpy="0 0 0" />
       </cylinder_inertial>
+      <!-- <inertial>
+        <mass value="8.393"/>
+        <inertia ixx="0.22689067591036" ixy="0.0" ixz="0.0" iyy="0.22689067591036" iyz="0.0" izz="0.0151074" />
+        <origin rpy="0.0 0.0 0.0" xyz="0.0 -0.024201 0.2125"/>
+      </inertial> -->
     </link>
     <!-- joint3 connects link2 and link3 -->
@@ -133,7 +150,8 @@
       <axis xyz="0 1 0" />
       <limit lower="-3.14" upper="3.14" effort="150.0" velocity="3.15" />
-      <dynamics damping="1" friction="1" />
+      <dynamics damping="1.0" />
     </joint>
     <!-- link 3 -->
+    <!-- forearm link -->
     <link name="ur5_link3">
       <visual>
@@ -153,4 +171,9 @@
         <origin xyz="0.0 0.0 0.25" rpy="0 0 0" />
       </cylinder_inertial>
+      <!-- <inertial>
+        <mass value="2.275"/>
+        <origin rpy="0.0 0.0 0.0" xyz="0.0 0.0265 0.11993"/>
+        <inertia ixx="0.049443313556" ixy="0.0" ixz="0.0" iyy="0.049443313556" iyz="0.0" izz="0.004095" />
+      </inertial> -->
     </link>
     <!-- joint4 connects link3 and link4 -->
@@ -161,5 +184,5 @@
       <axis xyz="0 1 0" />
       <limit lower="-3.14" upper="3.14" effort="28.0" velocity="3.2" />
-      <dynamics damping="1" friction="1" />
+      <dynamics damping="1.0" />
     </joint>
     <!-- link 4 -->
@@ -181,4 +204,9 @@
         <origin xyz="0.0 0.0 0.0" rpy="0 0 0" />
       </cylinder_inertial>
+      <!-- <inertial>
+        <mass value="1.219"/>
+        <origin rpy="0.0 0.0 0.0" xyz="0.0 0.110949 0.01634"/>
+        <inertia ixx="0.11117275553088" ixy="0.0" ixz="0.0" iyy="0.11117275553088" iyz="0.0" izz="0.21942" />
+      </inertial> -->
     </link>
     <!-- joint5 connects link4 and link5 -->
@@ -189,5 +217,5 @@
       <axis xyz="0 0 1" />
       <limit lower="-3.14" upper="3.14" effort="28.0" velocity="3.2" />
-      <dynamics damping="1" friction="1" />
+      <dynamics damping="1.0" />
     </joint>
     <!-- link 5 -->
@@ -209,4 +237,9 @@
         <origin xyz="0.0 0.0 0.0" rpy="0 0 0" />
       </cylinder_inertial>
+      <!-- <inertial>
+        <mass value="1.219"/>
+        <origin rpy="0.0 0.0 0.0" xyz="0.0 0.0018 0.11099"/>
+        <inertia ixx="0.11117275553088" ixy="0.0" ixz="0.0" iyy="0.11117275553088" iyz="0.0" izz="0.21942" />
+      </inertial> -->
     </link>
     <!-- joint6 connects link5 and link6 -->
@@ -217,5 +250,5 @@
       <axis xyz="0 1 0" />
       <limit lower="-3.14" upper="3.14" effort="28.0" velocity="3.2" />
-      <dynamics damping="1" friction="1" />
+      <dynamics damping="1.0" />
     </joint>
     <!-- link 6 -->
@@ -237,149 +270,10 @@
         <origin xyz="0.0 0.0 0.0" rpy="0 0 0" />
       </cylinder_inertial>
+      <!-- <inertial>
+        <mass value="0.1879"/>
+        <origin rpy="0.0 0.0 0.0" xyz="0.0 0.001159 0.0"/>
+        <inertia ixx="0.017136473145408" ixy="0.0" ixz="0.0" iyy="0.017136473145408" iyz="0.0" izz="0.033822" />
+      </inertial> -->
     </link>
   </macro>
-  <!-- This is where WSG50 begins -->
-  <joint name="ur5_ee_fixed_joint" type="fixed">
-    <parent link="ur5_link6" />
-    <child link="wsg_base" />
-    <origin xyz="0.0 ${wrist_3_length} 0.0" rpy="-${pi/2} 0.0 0.0" />
-  </joint>
-  <link name="wsg_base">
-    <inertial>
-      <mass value="0.01" />
-      <origin xyz="0 0 0" />
-      <inertia ixx="0.01" ixy="0.0" ixz="0.0" iyy="0.01" iyz="0.0" izz="0.01" />
-    </inertial>
-    <visual>
-      <origin xyz="0.0 0 0" rpy="0 0 0" />
-      <geometry>
-        <mesh filename="package://ur5_description/meshes/visual/WSG50_110.stl" scale="1 1 1" />
-      </geometry>
-      <material name="grey">
-        <color rgba="0.5 0.5 0.5 1" />
-      </material>
-    </visual>
-    <collision>
-      <origin xyz="0.0 0 0" rpy="0 0 0" />
-      <geometry>
-        <mesh filename="package://ur5_description/meshes/collision/WSG50_110.stl" scale="1 1 1" />
-      </geometry>
-    </collision>
-  </link>
-  <joint name="jointwsg_gripper_left" type="prismatic">
-    <limit lower="-0.055" upper="-0.0027" effort="100" velocity="100" />
-    <origin xyz="0 0 0" rpy="0 0 0" />
-    <parent link="wsg_base" />
-    <child link="wsg_gripper_left" />
-    <dynamics friction="1" damping="1" />
-    <axis xyz="1 0 0" />
-  </joint>
-  <link name="wsg_gripper_left">
-    <inertial>
-      <mass value="0.01" />
-      <origin xyz="0 0 0" />
-      <inertia ixx="0.01" ixy="0.0" ixz="0.0" iyy="0.01" iyz="0.0" izz="0.01" />
-    </inertial>
-    <visual>
-      <origin xyz="0.0 0 0" rpy="0 0 0" />
-      <geometry>
-        <mesh filename="package://ur5_description/meshes/visual/GUIDE_WSG50_110.stl" scale="0.001 0.001 0.001" />
-      </geometry>
-      <material name="black">
-        <color rgba="0 0 0 1" />
-      </material>
-    </visual>
-    <collision>
-      <origin xyz="0 0 0" rpy="0 0 0" />
-      <geometry>
-        <mesh filename="package://ur5_description/meshes/collision/GUIDE_WSG50_110.stl" scale="0.001 0.001 0.001" />
-      </geometry>
-    </collision>
-  </link>
-  <joint name="wsg_jointfinger_left" type="fixed">
-    <origin xyz="0 0 0.023" rpy="0 0 0" />
-    <parent link="wsg_gripper_left" />
-    <child link="wsg_finger_left" />
-    <axis xyz="1 0 0" />
-  </joint>
-  <link name="wsg_finger_left">
-    <inertial>
-      <mass value="0.01" />
-      <origin xyz="0 0 0" />
-      <inertia ixx="0.01" ixy="0.0" ixz="0.0" iyy="0.01" iyz="0.0" izz="0.01" />
-    </inertial>
-    <visual>
-      <origin xyz="0.0 0 0" rpy="0 0 0" />
-      <geometry>
-        <mesh filename="package://ur5_description/meshes/visual/WSG-FMF.stl" scale="0.001 0.001 0.001" />
-      </geometry>
-      <material name="black">
-        <color rgba="0 0 0 1" />
-      </material>
-    </visual>
-    <collision>
-      <origin xyz="0 0 0" rpy="0 0 0" />
-      <geometry>
-        <mesh filename="package://ur5_description/meshes/collision/WSG-FMF.stl" scale="0.001 0.001 0.001" />
-      </geometry>
-    </collision>
-  </link>
-  <joint name="jointwsg_gripper_right" type="prismatic">
-    <limit lower="0.0027" upper="0.055" effort="100" velocity="100" />
-    <origin xyz="0 0 0" rpy="0 0 3.14159" />
-    <parent link="wsg_base" />
-    <child link="wsg_gripper_right" />
-    <axis xyz="-1 0 0" />
-    <dynamics friction="1" damping="1" />
-  </joint>
-  <link name="wsg_gripper_right">
-    <inertial>
-      <mass value="0.01" />
-      <origin xyz="0 0 0" />
-      <inertia ixx="0.01" ixy="0.0" ixz="0.0" iyy="0.01" iyz="0.0" izz="0.01" />
-    </inertial>
-    <visual>
-      <origin xyz="0.0 0 0" rpy="0 0 0" />
-      <geometry>
-        <mesh filename="package://ur5_description/meshes/visual/GUIDE_WSG50_110.stl" scale="0.001 0.001 0.001" />
-      </geometry>
-      <material name="black">
-        <color rgba="0 0 0 1" />
-      </material>
-    </visual>
-    <collision>
-      <origin xyz="0 0 0" rpy="0 0 0" />
-      <geometry>
-        <mesh filename="package://ur5_description/meshes/collision/GUIDE_WSG50_110.stl" scale="0.001 0.001 0.001" />
-      </geometry>
-    </collision>
-  </link>
-  <joint name="wsg_jointfinger_right" type="fixed">
-    <origin xyz="0 0 0.023" rpy="0 0 0" />
-    <parent link="wsg_gripper_right" />
-    <child link="wsg_finger_right" />
-    <axis xyz="1 0 0" />
-  </joint>
-  <link name="wsg_finger_right">
-    <inertial>
-      <mass value="0.01" />
-      <origin xyz="0 0 0" />
-      <inertia ixx="0.01" ixy="0.0" ixz="0.0" iyy="0.01" iyz="0.0" izz="0.01" />
-    </inertial>
-    <visual>
-      <origin xyz="0.0 0 0" rpy="0 0 0" />
-      <geometry>
-        <mesh filename="package://ur5_description/meshes/visual/WSG-FMF.stl" scale="0.001 0.001 0.001" />
-      </geometry>
-      <material name="black">
-        <color rgba="0 0 0 1" />
-      </material>
-    </visual>
-    <collision>
-      <origin xyz="0 0 0" rpy="0 0 0" />
-      <geometry>
-        <mesh filename="package://ur5_description/meshes/collision/WSG-FMF.stl" scale="0.001 0.001 0.001" />
-      </geometry>
-    </collision>
-  </link>
 </robot>
